Commit message: implement fitness function

File: temp.urdf (robot description, URDF)
Before this commit: robot pepe, 9 links, 8 joints
Links:
- removed link 13
- removed link 15
- removed link 17
- removed link 22
- removed link 26
- removed link 28
- added link 12, mass 0.0025642893058701504; collision cylinder length=0.931342287061448 radius=0.029604239777924146; visual cylinder length=0.931342287061448 radius=0.029604239777924146
- added link 23, mass 0.03784257185920819; collision cylinder length=0.3762620677441708 radius=0.1789246460986148; visual cylinder length=0.3762620677441708 radius=0.1789246460986148
- added link 25, mass 0.03784257185920819; collision cylinder length=0.3762620677441708 radius=0.1789246460986148; visual cylinder length=0.3762620677441708 radius=0.1789246460986148
- link 0: mass 0.009220698730933933 -> 1.9092804905754177; geometry collision cylinder length=0.8592440908158552 radius=0.8410109571107248; visual cylinder length=0.8592440908158552 radius=0.8410109571107248
- link 11: mass 0.6128790045480625 -> 0.0025642893058701504; geometry collision cylinder length=0.931342287061448 radius=0.029604239777924146; visual cylinder length=0.931342287061448 radius=0.029604239777924146
- link 24: mass 0.9813470617207559 -> 0.03784257185920819; geometry collision cylinder length=0.3762620677441708 radius=0.1789246460986148; visual cylinder length=0.3762620677441708 radius=0.1789246460986148
Joints:
- removed joint 13_to_0
- removed joint 15_to_0
- removed joint 17_to_0
- removed joint 22_to_11
- removed joint 24_to_13
- removed joint 26_to_15
- removed joint 28_to_17
- added joint 12_to_0: type revolute, parent 0, child 12, origin xyz=0.17689580424762807 0.44069609796301823 0.7589384082652485 rpy=9.27053800106616 3.4702977233726573 0.3258792651083962, axis 0 0 1, limit lower=3.1415 upper=-3.1415 effort=1 velocity=1
- added joint 23_to_0: type revolute, parent 0, child 23, origin xyz=0.4994598277855792 0.3916007418430635 0.15798073054839057 rpy=10.11349457794136 5.402199333057146 1.9591320375952974, axis 0 0 1, limit lower=3.1415 upper=-3.1415 effort=1 velocity=1
- added joint 24_to_0: type revolute, parent 0, child 24, origin xyz=0.4994598277855792 0.3916007418430635 0.15798073054839057 rpy=12.6418682224267 5.402199333057146 1.9591320375952974, axis 0 0 1, limit lower=3.1415 upper=-3.1415 effort=1 velocity=1
- added joint 25_to_0: type revolute, parent 0, child 25, origin xyz=0.4994598277855792 0.3916007418430635 0.15798073054839057 rpy=15.17024186691204 5.402199333057146 1.9591320375952974, axis 0 0 1, limit lower=3.1415 upper=-3.1415 effort=1 velocity=1
- joint 11_to_0: axis 0 1 0 -> 0 0 1; origin xyz=0.24479507907470544 0.07448017766325798 0.7483182858441086 rpy=3.290938437377684 3.0299756248655987 4.850100364496203 -> xyz=0.17689580424762807 0.44069609796301823 0.7589384082652485 rpy=6.18035866737744 3.4702977233726573 0.3258792651083962
