Commit message: implement fitness function

File: test.urdf (robot description, URDF)
Before this commit: robot pepe, 17 links, 16 joints
Links:
- removed link 113
- removed link 15
- removed link 19
- removed link 210
- removed link 211
- removed link 212
- removed link 214
- removed link 215
- removed link 216
- removed link 24
- removed link 26
- removed link 27
- removed link 28
- added link 119, mass 1.9922967795459348; collision cylinder length=0.837333264099701 radius=0.8702677860285559; visual cylinder length=0.837333264099701 radius=0.8702677860285559
- added link 137, mass 1.9922967795459348; collision cylinder length=0.837333264099701 radius=0.8702677860285559; visual cylinder length=0.837333264099701 radius=0.8702677860285559
- added link 220, mass 0.2228649377207587; collision cylinder length=0.714050517116996 radius=0.31519655985894235; visual cylinder length=0.714050517116996 radius=0.31519655985894235
- added link 221, mass 0.2228649377207587; collision cylinder length=0.714050517116996 radius=0.31519655985894235; visual cylinder length=0.714050517116996 radius=0.31519655985894235
- added link 238, mass 0.2228649377207587; collision cylinder length=0.714050517116996 radius=0.31519655985894235; visual cylinder length=0.714050517116996 radius=0.31519655985894235
- added link 239, mass 0.2228649377207587; collision cylinder length=0.714050517116996 radius=0.31519655985894235; visual cylinder length=0.714050517116996 radius=0.31519655985894235
- added link 314, mass 0.05808897324191857; collision cylinder length=0.5749107634105123 radius=0.17933774059315555; visual cylinder length=0.5749107634105123 radius=0.17933774059315555
- added link 322, mass 0.05808897324191857; collision cylinder length=0.5749107634105123 radius=0.17933774059315555; visual cylinder length=0.5749107634105123 radius=0.17933774059315555
- added link 327, mass 0.05808897324191857; collision cylinder length=0.5749107634105123 radius=0.17933774059315555; visual cylinder length=0.5749107634105123 radius=0.17933774059315555
- added link 332, mass 0.05808897324191857; collision cylinder length=0.5749107634105123 radius=0.17933774059315555; visual cylinder length=0.5749107634105123 radius=0.17933774059315555
- added link 34, mass 0.05808897324191857; collision cylinder length=0.5749107634105123 radius=0.17933774059315555; visual cylinder length=0.5749107634105123 radius=0.17933774059315555
- added link 340, mass 0.05808897324191857; collision cylinder length=0.5749107634105123 radius=0.17933774059315555; visual cylinder length=0.5749107634105123 radius=0.17933774059315555
- added link 345, mass 0.05808897324191857; collision cylinder length=0.5749107634105123 radius=0.17933774059315555; visual cylinder length=0.5749107634105123 radius=0.17933774059315555
- added link 350, mass 0.05808897324191857; collision cylinder length=0.5749107634105123 radius=0.17933774059315555; visual cylinder length=0.5749107634105123 radius=0.17933774059315555
- added link 39, mass 0.05808897324191857; collision cylinder length=0.5749107634105123 radius=0.17933774059315555; visual cylinder length=0.5749107634105123 radius=0.17933774059315555
- added link 410, mass 0.037965458817956564; collision cylinder length=0.4090863269137367 radius=0.17187468212895696; visual cylinder length=0.4090863269137367 radius=0.17187468212895696
- added link 411, mass 0.037965458817956564; collision cylinder length=0.4090863269137367 radius=0.17187468212895696; visual cylinder length=0.4090863269137367 radius=0.17187468212895696
- added link 412, mass 0.037965458817956564; collision cylinder length=0.4090863269137367 radius=0.17187468212895696; visual cylinder length=0.4090863269137367 radius=0.17187468212895696
- added link 413, mass 0.037965458817956564; collision cylinder length=0.4090863269137367 radius=0.17187468212895696; visual cylinder length=0.4090863269137367 radius=0.17187468212895696
- added link 415, mass 0.037965458817956564; collision cylinder length=0.4090863269137367 radius=0.17187468212895696; visual cylinder length=0.4090863269137367 radius=0.17187468212895696
- added link 416, mass 0.037965458817956564; collision cylinder length=0.4090863269137367 radius=0.17187468212895696; visual cylinder length=0.4090863269137367 radius=0.17187468212895696
- added link 417, mass 0.037965458817956564; collision cylinder length=0.4090863269137367 radius=0.17187468212895696; visual cylinder length=0.4090863269137367 radius=0.17187468212895696
- added link 418, mass 0.037965458817956564; collision cylinder length=0.4090863269137367 radius=0.17187468212895696; visual cylinder length=0.4090863269137367 radius=0.17187468212895696
- added link 423, mass 0.037965458817956564; collision cylinder length=0.4090863269137367 radius=0.17187468212895696; visual cylinder length=0.4090863269137367 radius=0.17187468212895696
- added link 424, mass 0.037965458817956564; collision cylinder length=0.4090863269137367 radius=0.17187468212895696; visual cylinder length=0.4090863269137367 radius=0.17187468212895696
- added link 425, mass 0.037965458817956564; collision cylinder length=0.4090863269137367 radius=0.17187468212895696; visual cylinder length=0.4090863269137367 radius=0.17187468212895696
- added link 426, mass 0.037965458817956564; collision cylinder length=0.4090863269137367 radius=0.17187468212895696; visual cylinder length=0.4090863269137367 radius=0.17187468212895696
- added link 428, mass 0.037965458817956564; collision cylinder length=0.4090863269137367 radius=0.17187468212895696; visual cylinder length=0.4090863269137367 radius=0.17187468212895696
- added link 429, mass 0.037965458817956564; collision cylinder length=0.4090863269137367 radius=0.17187468212895696; visual cylinder length=0.4090863269137367 radius=0.17187468212895696
- added link 430, mass 0.037965458817956564; collision cylinder length=0.4090863269137367 radius=0.17187468212895696; visual cylinder length=0.4090863269137367 radius=0.17187468212895696
- added link 431, mass 0.037965458817956564; collision cylinder length=0.4090863269137367 radius=0.17187468212895696; visual cylinder length=0.4090863269137367 radius=0.17187468212895696
- added link 433, mass 0.037965458817956564; collision cylinder length=0.4090863269137367 radius=0.17187468212895696; visual cylinder length=0.4090863269137367 radius=0.17187468212895696
- added link 434, mass 0.037965458817956564; collision cylinder length=0.4090863269137367 radius=0.17187468212895696; visual cylinder length=0.4090863269137367 radius=0.17187468212895696
- added link 435, mass 0.037965458817956564; collision cylinder length=0.4090863269137367 radius=0.17187468212895696; visual cylinder length=0.4090863269137367 radius=0.17187468212895696
- added link 436, mass 0.037965458817956564; collision cylinder length=0.4090863269137367 radius=0.17187468212895696; visual cylinder length=0.4090863269137367 radius=0.17187468212895696
- added link 441, mass 0.037965458817956564; collision cylinder length=0.4090863269137367 radius=0.17187468212895696; visual cylinder length=0.4090863269137367 radius=0.17187468212895696
- added link 442, mass 0.037965458817956564; collision cylinder length=0.4090863269137367 radius=0.17187468212895696; visual cylinder length=0.4090863269137367 radius=0.17187468212895696
- added link 443, mass 0.037965458817956564; collision cylinder length=0.4090863269137367 radius=0.17187468212895696; visual cylinder length=0.4090863269137367 radius=0.17187468212895696
- added link 444, mass 0.037965458817956564; collision cylinder length=0.4090863269137367 radius=0.17187468212895696; visual cylinder length=0.4090863269137367 radius=0.17187468212895696
- added link 446, mass 0.037965458817956564; collision cylinder length=0.4090863269137367 radius=0.17187468212895696; visual cylinder length=0.4090863269137367 radius=0.17187468212895696
- added link 447, mass 0.037965458817956564; collision cylinder length=0.4090863269137367 radius=0.17187468212895696; visual cylinder length=0.4090863269137367 radius=0.17187468212895696
- added link 448, mass 0.037965458817956564; collision cylinder length=0.4090863269137367 radius=0.17187468212895696; visual cylinder length=0.4090863269137367 radius=0.17187468212895696
- added link 449, mass 0.037965458817956564; collision cylinder length=0.4090863269137367 radius=0.17187468212895696; visual cylinder length=0.4090863269137367 radius=0.17187468212895696
- added link 45, mass 0.037965458817956564; collision cylinder length=0.4090863269137367 radius=0.17187468212895696; visual cylinder length=0.4090863269137367 radius=0.17187468212895696
- added link 451, mass 0.037965458817956564; collision cylinder length=0.4090863269137367 radius=0.17187468212895696; visual cylinder length=0.4090863269137367 radius=0.17187468212895696
- added link 452, mass 0.037965458817956564; collision cylinder length=0.4090863269137367 radius=0.17187468212895696; visual cylinder length=0.4090863269137367 radius=0.17187468212895696
- added link 453, mass 0.037965458817956564; collision cylinder length=0.4090863269137367 radius=0.17187468212895696; visual cylinder length=0.4090863269137367 radius=0.17187468212895696
- added link 454, mass 0.037965458817956564; collision cylinder length=0.4090863269137367 radius=0.17187468212895696; visual cylinder length=0.4090863269137367 radius=0.17187468212895696
- added link 46, mass 0.037965458817956564; collision cylinder length=0.4090863269137367 radius=0.17187468212895696; visual cylinder length=0.4090863269137367 radius=0.17187468212895696
- added link 47, mass 0.037965458817956564; collision cylinder length=0.4090863269137367 radius=0.17187468212895696; visual cylinder length=0.4090863269137367 radius=0.17187468212895696
- added link 48, mass 0.037965458817956564; collision cylinder length=0.4090863269137367 radius=0.17187468212895696; visual cylinder length=0.4090863269137367 radius=0.17187468212895696
- link 0: mass 0.11117973710829591 -> 0.45752019238045055; geometry collision cylinder length=0.5956021415631482 radius=0.49448380381731394; visual cylinder length=0.5956021415631482 radius=0.49448380381731394
- link 11: mass 0.0003808477477781424 -> 1.9922967795459348; geometry collision cylinder length=0.837333264099701 radius=0.8702677860285559; visual cylinder length=0.837333264099701 radius=0.8702677860285559
- link 22: mass 0.16291732810421408 -> 0.2228649377207587; geometry collision cylinder length=0.714050517116996 radius=0.31519655985894235; visual cylinder length=0.714050517116996 radius=0.31519655985894235
- link 23: mass 0.16291732810421408 -> 0.2228649377207587; geometry collision cylinder length=0.714050517116996 radius=0.31519655985894235; visual cylinder length=0.714050517116996 radius=0.31519655985894235
Joints:
- removed joint 113_to_0
- removed joint 15_to_0
- removed joint 19_to_0
- removed joint 210_to_19
- removed joint 211_to_19
- removed joint 212_to_19
- removed joint 214_to_113
- removed joint 215_to_113
- removed joint 216_to_113
- removed joint 24_to_11
- removed joint 26_to_15
- removed joint 27_to_15
- removed joint 28_to_15
- added joint 119_to_0: type revolute, parent 0, child 119, origin xyz=0.35362981115640146 0.8849129081775543 0.08372428731370674 rpy=16.882540709097754 5.166318824637535 0.6942491317139261, axis 0 0 1, limit lower=3.1415 upper=-3.1415 effort=1 velocity=1
- added joint 137_to_0: type revolute, parent 0, child 137, origin xyz=0.35362981115640146 0.8849129081775543 0.08372428731370674 rpy=22.510054278797007 5.166318824637535 0.6942491317139261, axis 0 0 1, limit lower=3.1415 upper=-3.1415 effort=1 velocity=1
- added joint 220_to_119: type revolute, parent 119, child 220, origin xyz=0.3221595825928266 0.7552748145158681 0.294799539339191 rpy=1.812321266055931 3.8199719505239744 3.5480404510740544, axis 0 0 1, limit lower=3.1415 upper=-3.1415 effort=1 velocity=1
- added joint 221_to_119: type revolute, parent 119, child 221, origin xyz=0.3221595825928266 0.7552748145158681 0.294799539339191 rpy=2.7184818990838964 3.8199719505239744 3.5480404510740544, axis 0 0 1, limit lower=3.1415 upper=-3.1415 effort=1 velocity=1
- added joint 238_to_137: type revolute, parent 137, child 238, origin xyz=0.3221595825928266 0.7552748145158681 0.294799539339191 rpy=1.812321266055931 3.8199719505239744 3.5480404510740544, axis 0 0 1, limit lower=3.1415 upper=-3.1415 effort=1 velocity=1
- added joint 239_to_137: type revolute, parent 137, child 239, origin xyz=0.3221595825928266 0.7552748145158681 0.294799539339191 rpy=2.7184818990838964 3.8199719505239744 3.5480404510740544, axis 0 0 1, limit lower=3.1415 upper=-3.1415 effort=1 velocity=1
- added joint 314_to_11: type revolute, parent 11, child 314, origin xyz=0.3031068069905477 0.23727806236929283 0.686691103359021 rpy=0.37154126882008454 1.5961273355778953 6.254298719115715, axis 1 0 0, limit lower=3.1415 upper=-3.1415 effort=1 velocity=1
- added joint 322_to_119: type revolute, parent 119, child 322, origin xyz=0.3031068069905477 0.23727806236929283 0.686691103359021 rpy=0.24769417921338968 1.5961273355778953 6.254298719115715, axis 1 0 0, limit lower=3.1415 upper=-3.1415 effort=1 velocity=1
- added joint 327_to_119: type revolute, parent 119, child 327, origin xyz=0.3031068069905477 0.23727806236929283 0.686691103359021 rpy=0.3096177240167371 1.5961273355778953 6.254298719115715, axis 1 0 0, limit lower=3.1415 upper=-3.1415 effort=1 velocity=1
- added joint 332_to_119: type revolute, parent 119, child 332, origin xyz=0.3031068069905477 0.23727806236929283 0.686691103359021 rpy=0.37154126882008454 1.5961273355778953 6.254298719115715, axis 1 0 0, limit lower=3.1415 upper=-3.1415 effort=1 velocity=1
- added joint 340_to_137: type revolute, parent 137, child 340, origin xyz=0.3031068069905477 0.23727806236929283 0.686691103359021 rpy=0.24769417921338968 1.5961273355778953 6.254298719115715, axis 1 0 0, limit lower=3.1415 upper=-3.1415 effort=1 velocity=1
- added joint 345_to_137: type revolute, parent 137, child 345, origin xyz=0.3031068069905477 0.23727806236929283 0.686691103359021 rpy=0.3096177240167371 1.5961273355778953 6.254298719115715, axis 1 0 0, limit lower=3.1415 upper=-3.1415 effort=1 velocity=1
- added joint 34_to_11: type revolute, parent 11, child 34, origin xyz=0.3031068069905477 0.23727806236929283 0.686691103359021 rpy=0.24769417921338968 1.5961273355778953 6.254298719115715, axis 1 0 0, limit lower=3.1415 upper=-3.1415 effort=1 velocity=1
- added joint 350_to_137: type revolute, parent 137, child 350, origin xyz=0.3031068069905477 0.23727806236929283 0.686691103359021 rpy=0.37154126882008454 1.5961273355778953 6.254298719115715, axis 1 0 0, limit lower=3.1415 upper=-3.1415 effort=1 velocity=1
- added joint 39_to_11: type revolute, parent 11, child 39, origin xyz=0.3031068069905477 0.23727806236929283 0.686691103359021 rpy=0.3096177240167371 1.5961273355778953 6.254298719115715, axis 1 0 0, limit lower=3.1415 upper=-3.1415 effort=1 velocity=1
- added joint 410_to_39: type revolute, parent 39, child 410, origin xyz=0.7171330316248481 0.3632760327971024 0.05485458015927103 rpy=5.630593456049959 0.7025410358322909 1.8355683681169181, axis 0 0 1, limit lower=3.1415 upper=-3.1415 effort=1 velocity=1
- added joint 411_to_39: type revolute, parent 39, child 411, origin xyz=0.7171330316248481 0.3632760327971024 0.05485458015927103 rpy=8.445890184074939 0.7025410358322909 1.8355683681169181, axis 0 0 1, limit lower=3.1415 upper=-3.1415 effort=1 velocity=1
- added joint 412_to_39: type revolute, parent 39, child 412, origin xyz=0.7171330316248481 0.3632760327971024 0.05485458015927103 rpy=11.261186912099918 0.7025410358322909 1.8355683681169181, axis 0 0 1, limit lower=3.1415 upper=-3.1415 effort=1 velocity=1
- added joint 413_to_39: type revolute, parent 39, child 413, origin xyz=0.7171330316248481 0.3632760327971024 0.05485458015927103 rpy=14.076483640124897 0.7025410358322909 1.8355683681169181, axis 0 0 1, limit lower=3.1415 upper=-3.1415 effort=1 velocity=1
- added joint 415_to_314: type revolute, parent 314, child 415, origin xyz=0.7171330316248481 0.3632760327971024 0.05485458015927103 rpy=5.630593456049959 0.7025410358322909 1.8355683681169181, axis 0 0 1, limit lower=3.1415 upper=-3.1415 effort=1 velocity=1
- added joint 416_to_314: type revolute, parent 314, child 416, origin xyz=0.7171330316248481 0.3632760327971024 0.05485458015927103 rpy=8.445890184074939 0.7025410358322909 1.8355683681169181, axis 0 0 1, limit lower=3.1415 upper=-3.1415 effort=1 velocity=1
- added joint 417_to_314: type revolute, parent 314, child 417, origin xyz=0.7171330316248481 0.3632760327971024 0.05485458015927103 rpy=11.261186912099918 0.7025410358322909 1.8355683681169181, axis 0 0 1, limit lower=3.1415 upper=-3.1415 effort=1 velocity=1
- added joint 418_to_314: type revolute, parent 314, child 418, origin xyz=0.7171330316248481 0.3632760327971024 0.05485458015927103 rpy=14.076483640124897 0.7025410358322909 1.8355683681169181, axis 0 0 1, limit lower=3.1415 upper=-3.1415 effort=1 velocity=1
- added joint 423_to_322: type revolute, parent 322, child 423, origin xyz=0.7171330316248481 0.3632760327971024 0.05485458015927103 rpy=5.630593456049959 0.7025410358322909 1.8355683681169181, axis 0 0 1, limit lower=3.1415 upper=-3.1415 effort=1 velocity=1
- added joint 424_to_322: type revolute, parent 322, child 424, origin xyz=0.7171330316248481 0.3632760327971024 0.05485458015927103 rpy=8.445890184074939 0.7025410358322909 1.8355683681169181, axis 0 0 1, limit lower=3.1415 upper=-3.1415 effort=1 velocity=1
- added joint 425_to_322: type revolute, parent 322, child 425, origin xyz=0.7171330316248481 0.3632760327971024 0.05485458015927103 rpy=11.261186912099918 0.7025410358322909 1.8355683681169181, axis 0 0 1, limit lower=3.1415 upper=-3.1415 effort=1 velocity=1
- added joint 426_to_322: type revolute, parent 322, child 426, origin xyz=0.7171330316248481 0.3632760327971024 0.05485458015927103 rpy=14.076483640124897 0.7025410358322909 1.8355683681169181, axis 0 0 1, limit lower=3.1415 upper=-3.1415 effort=1 velocity=1
- added joint 428_to_327: type revolute, parent 327, child 428, origin xyz=0.7171330316248481 0.3632760327971024 0.05485458015927103 rpy=5.630593456049959 0.7025410358322909 1.8355683681169181, axis 0 0 1, limit lower=3.1415 upper=-3.1415 effort=1 velocity=1
- added joint 429_to_327: type revolute, parent 327, child 429, origin xyz=0.7171330316248481 0.3632760327971024 0.05485458015927103 rpy=8.445890184074939 0.7025410358322909 1.8355683681169181, axis 0 0 1, limit lower=3.1415 upper=-3.1415 effort=1 velocity=1
- added joint 430_to_327: type revolute, parent 327, child 430, origin xyz=0.7171330316248481 0.3632760327971024 0.05485458015927103 rpy=11.261186912099918 0.7025410358322909 1.8355683681169181, axis 0 0 1, limit lower=3.1415 upper=-3.1415 effort=1 velocity=1
- added joint 431_to_327: type revolute, parent 327, child 431, origin xyz=0.7171330316248481 0.3632760327971024 0.05485458015927103 rpy=14.076483640124897 0.7025410358322909 1.8355683681169181, axis 0 0 1, limit lower=3.1415 upper=-3.1415 effort=1 velocity=1
- added joint 433_to_332: type revolute, parent 332, child 433, origin xyz=0.7171330316248481 0.3632760327971024 0.05485458015927103 rpy=5.630593456049959 0.7025410358322909 1.8355683681169181, axis 0 0 1, limit lower=3.1415 upper=-3.1415 effort=1 velocity=1
- added joint 434_to_332: type revolute, parent 332, child 434, origin xyz=0.7171330316248481 0.3632760327971024 0.05485458015927103 rpy=8.445890184074939 0.7025410358322909 1.8355683681169181, axis 0 0 1, limit lower=3.1415 upper=-3.1415 effort=1 velocity=1
- added joint 435_to_332: type revolute, parent 332, child 435, origin xyz=0.7171330316248481 0.3632760327971024 0.05485458015927103 rpy=11.261186912099918 0.7025410358322909 1.8355683681169181, axis 0 0 1, limit lower=3.1415 upper=-3.1415 effort=1 velocity=1
- added joint 436_to_332: type revolute, parent 332, child 436, origin xyz=0.7171330316248481 0.3632760327971024 0.05485458015927103 rpy=14.076483640124897 0.7025410358322909 1.8355683681169181, axis 0 0 1, limit lower=3.1415 upper=-3.1415 effort=1 velocity=1
- added joint 441_to_340: type revolute, parent 340, child 441, origin xyz=0.7171330316248481 0.3632760327971024 0.05485458015927103 rpy=5.630593456049959 0.7025410358322909 1.8355683681169181, axis 0 0 1, limit lower=3.1415 upper=-3.1415 effort=1 velocity=1
- added joint 442_to_340: type revolute, parent 340, child 442, origin xyz=0.7171330316248481 0.3632760327971024 0.05485458015927103 rpy=8.445890184074939 0.7025410358322909 1.8355683681169181, axis 0 0 1, limit lower=3.1415 upper=-3.1415 effort=1 velocity=1
- added joint 443_to_340: type revolute, parent 340, child 443, origin xyz=0.7171330316248481 0.3632760327971024 0.05485458015927103 rpy=11.261186912099918 0.7025410358322909 1.8355683681169181, axis 0 0 1, limit lower=3.1415 upper=-3.1415 effort=1 velocity=1
- added joint 444_to_340: type revolute, parent 340, child 444, origin xyz=0.7171330316248481 0.3632760327971024 0.05485458015927103 rpy=14.076483640124897 0.7025410358322909 1.8355683681169181, axis 0 0 1, limit lower=3.1415 upper=-3.1415 effort=1 velocity=1
- added joint 446_to_345: type revolute, parent 345, child 446, origin xyz=0.7171330316248481 0.3632760327971024 0.05485458015927103 rpy=5.630593456049959 0.7025410358322909 1.8355683681169181, axis 0 0 1, limit lower=3.1415 upper=-3.1415 effort=1 velocity=1
- added joint 447_to_345: type revolute, parent 345, child 447, origin xyz=0.7171330316248481 0.3632760327971024 0.05485458015927103 rpy=8.445890184074939 0.7025410358322909 1.8355683681169181, axis 0 0 1, limit lower=3.1415 upper=-3.1415 effort=1 velocity=1
- added joint 448_to_345: type revolute, parent 345, child 448, origin xyz=0.7171330316248481 0.3632760327971024 0.05485458015927103 rpy=11.261186912099918 0.7025410358322909 1.8355683681169181, axis 0 0 1, limit lower=3.1415 upper=-3.1415 effort=1 velocity=1
- added joint 449_to_345: type revolute, parent 345, child 449, origin xyz=0.7171330316248481 0.3632760327971024 0.05485458015927103 rpy=14.076483640124897 0.7025410358322909 1.8355683681169181, axis 0 0 1, limit lower=3.1415 upper=-3.1415 effort=1 velocity=1
- added joint 451_to_350: type revolute, parent 350, child 451, origin xyz=0.7171330316248481 0.3632760327971024 0.05485458015927103 rpy=5.630593456049959 0.7025410358322909 1.8355683681169181, axis 0 0 1, limit lower=3.1415 upper=-3.1415 effort=1 velocity=1
- added joint 452_to_350: type revolute, parent 350, child 452, origin xyz=0.7171330316248481 0.3632760327971024 0.05485458015927103 rpy=8.445890184074939 0.7025410358322909 1.8355683681169181, axis 0 0 1, limit lower=3.1415 upper=-3.1415 effort=1 velocity=1
- added joint 453_to_350: type revolute, parent 350, child 453, origin xyz=0.7171330316248481 0.3632760327971024 0.05485458015927103 rpy=11.261186912099918 0.7025410358322909 1.8355683681169181, axis 0 0 1, limit lower=3.1415 upper=-3.1415 effort=1 velocity=1
- added joint 454_to_350: type revolute, parent 350, child 454, origin xyz=0.7171330316248481 0.3632760327971024 0.05485458015927103 rpy=14.076483640124897 0.7025410358322909 1.8355683681169181, axis 0 0 1, limit lower=3.1415 upper=-3.1415 effort=1 velocity=1
- added joint 45_to_34: type revolute, parent 34, child 45, origin xyz=0.7171330316248481 0.3632760327971024 0.05485458015927103 rpy=5.630593456049959 0.7025410358322909 1.8355683681169181, axis 0 0 1, limit lower=3.1415 upper=-3.1415 effort=1 velocity=1
- added joint 46_to_34: type revolute, parent 34, child 46, origin xyz=0.7171330316248481 0.3632760327971024 0.05485458015927103 rpy=8.445890184074939 0.7025410358322909 1.8355683681169181, axis 0 0 1, limit lower=3.1415 upper=-3.1415 effort=1 velocity=1
- added joint 47_to_34: type revolute, parent 34, child 47, origin xyz=0.7171330316248481 0.3632760327971024 0.05485458015927103 rpy=11.261186912099918 0.7025410358322909 1.8355683681169181, axis 0 0 1, limit lower=3.1415 upper=-3.1415 effort=1 velocity=1
- added joint 48_to_34: type revolute, parent 34, child 48, origin xyz=0.7171330316248481 0.3632760327971024 0.05485458015927103 rpy=14.076483640124897 0.7025410358322909 1.8355683681169181, axis 0 0 1, limit lower=3.1415 upper=-3.1415 effort=1 velocity=1
- joint 11_to_0: axis 0 1 0 -> 0 0 1; origin xyz=0.588360315768213 0.7144939802055135 0.8759301769331351 rpy=4.791569022126908 3.3803455565831606 3.360197768605905 -> xyz=0.35362981115640146 0.8849129081775543 0.08372428731370674 rpy=11.255027139398504 5.166318824637535 0.6942491317139261
- joint 22_to_11: axis 0 1 0 -> 0 0 1; origin xyz=0.534221713157885 0.7572050361852153 0.21156947154303396 rpy=11.828824807098005 2.4235413610076293 1.0289950641395593 -> xyz=0.3221595825928266 0.7552748145158681 0.294799539339191 rpy=1.812321266055931 3.8199719505239744 3.5480404510740544
- joint 23_to_11: axis 0 1 0 -> 0 0 1; origin xyz=0.534221713157885 0.7572050361852153 0.21156947154303396 rpy=17.74323721064701 2.4235413610076293 1.0289950641395593 -> xyz=0.3221595825928266 0.7552748145158681 0.294799539339191 rpy=2.7184818990838964 3.8199719505239744 3.5480404510740544
