Commit message: implement genetic algorithm with evolution

File: temp2.urdf (robot description, URDF)
Before this commit: robot pepe, 9 links, 8 joints
Links:
- removed link 15
- removed link 17
- removed link 22
- removed link 24
- removed link 26
- removed link 28
- added link 12, mass 2.0050681046279117; collision cylinder length=0.6893211687453101 radius=0.9622298383937432; visual cylinder length=0.6893211687453101 radius=0.9622298383937432
- added link 14, mass 2.0050681046279117; collision cylinder length=0.6893211687453101 radius=0.9622298383937432; visual cylinder length=0.6893211687453101 radius=0.9622298383937432
- link 0: mass 2.7523101715011373 -> 0.6712655145949162; geometry collision cylinder length=0.637638808771346 radius=0.5788750892855647; visual cylinder length=0.637638808771346 radius=0.5788750892855647
- link 11: mass 0.1160743071039241 -> 2.0050681046279117; geometry collision cylinder length=0.6893211687453101 radius=0.9622298383937432; visual cylinder length=0.6893211687453101 radius=0.9622298383937432
- link 13: mass 0.1160743071039241 -> 2.0050681046279117; geometry collision cylinder length=0.6893211687453101 radius=0.9622298383937432; visual cylinder length=0.6893211687453101 radius=0.9622298383937432
Joints:
- removed joint 15_to_0
- removed joint 17_to_0
- removed joint 22_to_11
- removed joint 24_to_13
- removed joint 26_to_15
- removed joint 28_to_17
- added joint 12_to_0: type revolute, parent 0, child 12, origin xyz=0.7089214976795559 0.8965713998574288 0.9739570469538621 rpy=15.064248610142968 0.25339753699709533 2.2338164889001972, axis 0 1 0, limit lower=3.1415 upper=-3.1415 effort=1 velocity=1
- added joint 14_to_0: type revolute, parent 0, child 14, origin xyz=0.7089214976795559 0.8965713998574288 0.9739570469538621 rpy=25.10708101690495 0.25339753699709533 2.2338164889001972, axis 0 1 0, limit lower=3.1415 upper=-3.1415 effort=1 velocity=1
- joint 11_to_0: origin xyz=0.6272106166922962 0.21176605765536027 0.4480087464323598 rpy=5.279768773702489 5.33341798195908 2.427282067818647 -> xyz=0.7089214976795559 0.8965713998574288 0.9739570469538621 rpy=10.04283240676198 0.25339753699709533 2.2338164889001972
- joint 13_to_0: origin xyz=0.6272106166922962 0.21176605765536027 0.4480087464323598 rpy=7.919653160553734 5.33341798195908 2.427282067818647 -> xyz=0.7089214976795559 0.8965713998574288 0.9739570469538621 rpy=20.08566481352396 0.25339753699709533 2.2338164889001972

File: temp3.urdf (robot description, URDF)
Before this commit: robot pepe, 9 links, 8 joints
Links:
- removed link 15
- removed link 22
- removed link 23
- removed link 24
- removed link 28
- added link 12, mass 2.0050681046279117; collision cylinder length=0.6893211687453101 radius=0.9622298383937432; visual cylinder length=0.6893211687453101 radius=0.9622298383937432
- added link 13, mass 2.0050681046279117; collision cylinder length=0.6893211687453101 radius=0.9622298383937432; visual cylinder length=0.6893211687453101 radius=0.9622298383937432
- added link 14, mass 2.0050681046279117; collision cylinder length=0.6893211687453101 radius=0.9622298383937432; visual cylinder length=0.6893211687453101 radius=0.9622298383937432
- added link 25, mass 0.9083716675679936; collision cylinder length=0.8910416748445856 radius=0.569649663536754; visual cylinder length=0.8910416748445856 radius=0.569649663536754
- link 0: mass 0.9694459477196559 -> 0.6712655145949162; geometry collision cylinder length=0.637638808771346 radius=0.5788750892855647; visual cylinder length=0.637638808771346 radius=0.5788750892855647
- link 11: mass 1.6390072666514175 -> 2.0050681046279117; geometry collision cylinder length=0.6893211687453101 radius=0.9622298383937432; visual cylinder length=0.6893211687453101 radius=0.9622298383937432
- link 26: mass 0.03867159938222178 -> 0.9083716675679936; geometry collision cylinder length=0.8910416748445856 radius=0.569649663536754; visual cylinder length=0.8910416748445856 radius=0.569649663536754
- link 27: mass 0.03867159938222178 -> 0.9083716675679936; geometry collision cylinder length=0.8910416748445856 radius=0.569649663536754; visual cylinder length=0.8910416748445856 radius=0.569649663536754
Joints:
- removed joint 15_to_0
- removed joint 22_to_11
- removed joint 23_to_11
- removed joint 24_to_11
- removed joint 26_to_15
- removed joint 27_to_15
- removed joint 28_to_15
- added joint 12_to_0: type revolute, parent 0, child 12, origin xyz=0.7089214976795559 0.8965713998574288 0.9739570469538621 rpy=15.064248610142968 0.25339753699709533 2.2338164889001972, axis 0 1 0, limit lower=3.1415 upper=-3.1415 effort=1 velocity=1
- added joint 13_to_0: type revolute, parent 0, child 13, origin xyz=0.7089214976795559 0.8965713998574288 0.9739570469538621 rpy=20.08566481352396 0.25339753699709533 2.2338164889001972, axis 0 1 0, limit lower=3.1415 upper=-3.1415 effort=1 velocity=1
- added joint 14_to_0: type revolute, parent 0, child 14, origin xyz=0.7089214976795559 0.8965713998574288 0.9739570469538621 rpy=25.10708101690495 0.25339753699709533 2.2338164889001972, axis 0 1 0, limit lower=3.1415 upper=-3.1415 effort=1 velocity=1
- added joint 25_to_0: type revolute, parent 0, child 25, origin xyz=0.08216211729265621 0.6579921822788458 0.5292909840462087 rpy=16.966224225645128 2.0248785601380037 4.606704575895256, axis 0 0 1, limit lower=3.1415 upper=-3.1415 effort=1 velocity=1
- added joint 26_to_0: type revolute, parent 0, child 26, origin xyz=0.08216211729265621 0.6579921822788458 0.5292909840462087 rpy=19.79392826325265 2.0248785601380037 4.606704575895256, axis 0 0 1, limit lower=3.1415 upper=-3.1415 effort=1 velocity=1
- added joint 27_to_0: type revolute, parent 0, child 27, origin xyz=0.08216211729265621 0.6579921822788458 0.5292909840462087 rpy=22.62163230086017 2.0248785601380037 4.606704575895256, axis 0 0 1, limit lower=3.1415 upper=-3.1415 effort=1 velocity=1
- joint 11_to_0: origin xyz=0.11735432136907897 0.01201470122286541 0.3395072903966563 rpy=7.219679045886174 5.062294171260698 5.014112013523304 -> xyz=0.7089214976795559 0.8965713998574288 0.9739570469538621 rpy=10.04283240676198 0.25339753699709533 2.2338164889001972

File: temp7.urdf (robot description, URDF)
Before this commit: robot pepe, 3 links, 2 joints
Links:
- removed link 12
- added link 13, mass 0.37533349993301535; collision cylinder length=0.24563081295102152 radius=0.6974166398949238; visual cylinder length=0.24563081295102152 radius=0.6974166398949238
- added link 22, mass 0.23470184442502104; collision cylinder length=0.6782894717223117 radius=0.3318759463979437; visual cylinder length=0.6782894717223117 radius=0.3318759463979437
- added link 24, mass 0.23470184442502104; collision cylinder length=0.6782894717223117 radius=0.3318759463979437; visual cylinder length=0.6782894717223117 radius=0.3318759463979437
Joints:
- removed joint 12_to_0
- added joint 13_to_0: type revolute, parent 0, child 13, origin xyz=0.3291841544527887 0.004449061513461916 0.18566610202390488 rpy=12.66331195587527 5.289662239770561 5.720727623375437, axis 0 0 1, limit lower=3.1415 upper=-3.1415 effort=1 velocity=1
- added joint 22_to_11: type revolute, parent 11, child 22, origin xyz=0.16796472666974804 0.9934904119759171 0.16790918914819897 rpy=2.5684511451391243 5.063506364403056 0.33076520107912166, axis 1 0 0, limit lower=3.1415 upper=-3.1415 effort=1 velocity=1
- added joint 24_to_13: type revolute, parent 13, child 24, origin xyz=0.16796472666974804 0.9934904119759171 0.16790918914819897 rpy=2.5684511451391243 5.063506364403056 0.33076520107912166, axis 1 0 0, limit lower=3.1415 upper=-3.1415 effort=1 velocity=1
