Commit message: add motor test script

File: test.urdf (robot description, URDF)
Before this commit: robot pepe, 221 links, 220 joints
Links:
- removed link 10201
- removed link 10202
- removed link 10203
- removed link 10204
- removed link 10206
- removed link 10207
- removed link 10208
- removed link 10209
- removed link 10211
- removed link 10212
- removed link 10213
- removed link 10214
- removed link 10216
- removed link 10217
- removed link 10218
- removed link 10219
- removed link 1114
- removed link 1115
- removed link 1116
- removed link 1122
- removed link 1123
- removed link 1124
- removed link 1130
- removed link 1131
- removed link 1132
- removed link 12101
- removed link 12106
- removed link 12117
- removed link 12122
- removed link 12127
- removed link 12132
- removed link 12142
- removed link 12147
- removed link 12152
- removed link 12157
- removed link 12167
- removed link 12172
- removed link 12177
- removed link 12182
- removed link 1241
- removed link 1246
- removed link 1251
- removed link 1256
- removed link 1266
- removed link 1271
- removed link 1276
- removed link 1281
- removed link 1291
- removed link 1296
- removed link 13191
- removed link 13192
- removed link 13193
- removed link 13194
- removed link 13196
- removed link 13197
- removed link 13198
- removed link 13199
- removed link 14111
- removed link 14112
- removed link 14137
- removed link 14138
- removed link 14162
- removed link 14163
- removed link 14187
- removed link 14188
- removed link 1461
- removed link 1462
- removed link 1486
- removed link 1487
- removed link 1511
- removed link 153
- removed link 157
- removed link 16100
- removed link 16102
- removed link 16103
- removed link 16104
- removed link 16105
- removed link 16107
- removed link 16108
- removed link 16109
- removed link 16110
- removed link 16118
- removed link 16119
- removed link 16120
- removed link 16121
- removed link 16123
- removed link 16124
- removed link 16125
- removed link 16126
- removed link 16128
- removed link 16129
- removed link 16130
- removed link 16131
- removed link 16133
- removed link 16134
- removed link 16135
- removed link 16136
- removed link 16143
- removed link 16144
- removed link 16145
- removed link 16146
- removed link 16148
- removed link 16149
- removed link 16150
- removed link 16151
- removed link 16153
- removed link 16154
- removed link 16155
- removed link 16156
- removed link 16158
- removed link 16159
- removed link 16160
- removed link 16161
- removed link 16168
- removed link 16169
- removed link 16170
- removed link 16171
- removed link 16173
- removed link 16174
- removed link 16175
- removed link 16176
- removed link 16178
- removed link 16179
- removed link 16180
- removed link 16181
- removed link 16183
- removed link 16184
- removed link 16185
- removed link 16186
- removed link 1642
- removed link 1643
- removed link 1644
- removed link 1645
- removed link 1647
- removed link 1648
- removed link 1649
- removed link 1650
- removed link 1652
- removed link 1653
- removed link 1654
- removed link 1655
- removed link 1657
- removed link 1658
- removed link 1659
- removed link 1660
- removed link 1667
- removed link 1668
- removed link 1669
- removed link 1670
- removed link 1672
- removed link 1673
- removed link 1674
- removed link 1675
- removed link 1677
- removed link 1678
- removed link 1679
- removed link 1680
- removed link 1682
- removed link 1683
- removed link 1684
- removed link 1685
- removed link 1692
- removed link 1693
- removed link 1694
- removed link 1695
- removed link 1697
- removed link 1698
- removed link 1699
- removed link 1712
- removed link 174
- removed link 178
- removed link 18220
- removed link 1917
- removed link 1918
- removed link 1919
- removed link 1920
- removed link 1925
- removed link 1926
- removed link 1927
- removed link 1928
- removed link 1933
- removed link 1934
- removed link 1935
- removed link 1936
- removed link 213
- removed link 221
- removed link 229
- removed link 3113
- removed link 337
- removed link 4114
- removed link 4139
- removed link 4164
- removed link 438
- removed link 463
- removed link 488
- removed link 510
- removed link 52
- removed link 56
- removed link 6115
- removed link 6116
- removed link 6140
- removed link 6141
- removed link 6165
- removed link 6166
- removed link 639
- removed link 640
- removed link 664
- removed link 665
- removed link 689
- removed link 690
- removed link 7189
- removed link 8190
- removed link 8195
- removed link 9200
- removed link 9205
- removed link 9210
- removed link 9215
- added link 113, mass 0.0003808477477781424; collision cylinder length=0.2987924817564709 radius=0.020142618472887786; visual cylinder length=0.2987924817564709 radius=0.020142618472887786
- added link 210, mass 0.16291732810421408; collision cylinder length=0.3959276825356993 radius=0.3619101548493394; visual cylinder length=0.3959276825356993 radius=0.3619101548493394
- added link 211, mass 0.16291732810421408; collision cylinder length=0.3959276825356993 radius=0.3619101548493394; visual cylinder length=0.3959276825356993 radius=0.3619101548493394
- added link 212, mass 0.16291732810421408; collision cylinder length=0.3959276825356993 radius=0.3619101548493394; visual cylinder length=0.3959276825356993 radius=0.3619101548493394
- added link 214, mass 0.16291732810421408; collision cylinder length=0.3959276825356993 radius=0.3619101548493394; visual cylinder length=0.3959276825356993 radius=0.3619101548493394
- added link 215, mass 0.16291732810421408; collision cylinder length=0.3959276825356993 radius=0.3619101548493394; visual cylinder length=0.3959276825356993 radius=0.3619101548493394
- added link 216, mass 0.16291732810421408; collision cylinder length=0.3959276825356993 radius=0.3619101548493394; visual cylinder length=0.3959276825356993 radius=0.3619101548493394
- added link 22, mass 0.16291732810421408; collision cylinder length=0.3959276825356993 radius=0.3619101548493394; visual cylinder length=0.3959276825356993 radius=0.3619101548493394
- added link 23, mass 0.16291732810421408; collision cylinder length=0.3959276825356993 radius=0.3619101548493394; visual cylinder length=0.3959276825356993 radius=0.3619101548493394
- added link 24, mass 0.16291732810421408; collision cylinder length=0.3959276825356993 radius=0.3619101548493394; visual cylinder length=0.3959276825356993 radius=0.3619101548493394
- added link 26, mass 0.16291732810421408; collision cylinder length=0.3959276825356993 radius=0.3619101548493394; visual cylinder length=0.3959276825356993 radius=0.3619101548493394
- added link 27, mass 0.16291732810421408; collision cylinder length=0.3959276825356993 radius=0.3619101548493394; visual cylinder length=0.3959276825356993 radius=0.3619101548493394
- added link 28, mass 0.16291732810421408; collision cylinder length=0.3959276825356993 radius=0.3619101548493394; visual cylinder length=0.3959276825356993 radius=0.3619101548493394
- link 0: mass 0.5610761225952888 -> 0.11117973710829591; geometry collision cylinder length=0.6875185842814737 radius=0.22687971294401033; visual cylinder length=0.6875185842814737 radius=0.22687971294401033
- link 11: mass 0.26493765993955554 -> 0.0003808477477781424; geometry collision cylinder length=0.2987924817564709 radius=0.020142618472887786; visual cylinder length=0.2987924817564709 radius=0.020142618472887786
- link 15: mass 0.26493765993955554 -> 0.0003808477477781424; geometry collision cylinder length=0.2987924817564709 radius=0.020142618472887786; visual cylinder length=0.2987924817564709 radius=0.020142618472887786
- link 19: mass 0.26493765993955554 -> 0.0003808477477781424; geometry collision cylinder length=0.2987924817564709 radius=0.020142618472887786; visual cylinder length=0.2987924817564709 radius=0.020142618472887786
Joints:
- removed joint 10201_to_9200
- removed joint 10202_to_9200
- removed joint 10203_to_9200
- removed joint 10204_to_9200
- removed joint 10206_to_9205
- removed joint 10207_to_9205
- removed joint 10208_to_9205
- removed joint 10209_to_9205
- removed joint 10211_to_9210
- removed joint 10212_to_9210
- removed joint 10213_to_9210
- removed joint 10214_to_9210
- removed joint 10216_to_9215
- removed joint 10217_to_9215
- removed joint 10218_to_9215
- removed joint 10219_to_9215
- removed joint 1114_to_213
- removed joint 1115_to_213
- removed joint 1116_to_213
- removed joint 1122_to_221
- removed joint 1123_to_221
- removed joint 1124_to_221
- removed joint 1130_to_229
- removed joint 1131_to_229
- removed joint 1132_to_229
- removed joint 12101_to_488
- removed joint 12106_to_488
- removed joint 12117_to_4114
- removed joint 12122_to_4114
- removed joint 12127_to_4114
- removed joint 12132_to_4114
- removed joint 12142_to_4139
- removed joint 12147_to_4139
- removed joint 12152_to_4139
- removed joint 12157_to_4139
- removed joint 12167_to_4164
- removed joint 12172_to_4164
- removed joint 12177_to_4164
- removed joint 12182_to_4164
- removed joint 1241_to_438
- removed joint 1246_to_438
- removed joint 1251_to_438
- removed joint 1256_to_438
- removed joint 1266_to_463
- removed joint 1271_to_463
- removed joint 1276_to_463
- removed joint 1281_to_463
- removed joint 1291_to_488
- removed joint 1296_to_488
- removed joint 13191_to_8190
- removed joint 13192_to_8190
- removed joint 13193_to_8190
- removed joint 13194_to_8190
- removed joint 13196_to_8195
- removed joint 13197_to_8195
- removed joint 13198_to_8195
- removed joint 13199_to_8195
- removed joint 14111_to_488
- removed joint 14112_to_488
- removed joint 14137_to_4114
- removed joint 14138_to_4114
- removed joint 14162_to_4139
- removed joint 14163_to_4139
- removed joint 14187_to_4164
- removed joint 14188_to_4164
- removed joint 1461_to_438
- removed joint 1462_to_438
- removed joint 1486_to_463
- removed joint 1487_to_463
- removed joint 1511_to_510
- removed joint 153_to_52
- removed joint 157_to_56
- removed joint 16100_to_1296
- removed joint 16102_to_12101
- removed joint 16103_to_12101
- removed joint 16104_to_12101
- removed joint 16105_to_12101
- removed joint 16107_to_12106
- removed joint 16108_to_12106
- removed joint 16109_to_12106
- removed joint 16110_to_12106
- removed joint 16118_to_12117
- removed joint 16119_to_12117
- removed joint 16120_to_12117
- removed joint 16121_to_12117
- removed joint 16123_to_12122
- removed joint 16124_to_12122
- removed joint 16125_to_12122
- removed joint 16126_to_12122
- removed joint 16128_to_12127
- removed joint 16129_to_12127
- removed joint 16130_to_12127
- removed joint 16131_to_12127
- removed joint 16133_to_12132
- removed joint 16134_to_12132
- removed joint 16135_to_12132
- removed joint 16136_to_12132
- removed joint 16143_to_12142
- removed joint 16144_to_12142
- removed joint 16145_to_12142
- removed joint 16146_to_12142
- removed joint 16148_to_12147
- removed joint 16149_to_12147
- removed joint 16150_to_12147
- removed joint 16151_to_12147
- removed joint 16153_to_12152
- removed joint 16154_to_12152
- removed joint 16155_to_12152
- removed joint 16156_to_12152
- removed joint 16158_to_12157
- removed joint 16159_to_12157
- removed joint 16160_to_12157
- removed joint 16161_to_12157
- removed joint 16168_to_12167
- removed joint 16169_to_12167
- removed joint 16170_to_12167
- removed joint 16171_to_12167
- removed joint 16173_to_12172
- removed joint 16174_to_12172
- removed joint 16175_to_12172
- removed joint 16176_to_12172
- removed joint 16178_to_12177
- removed joint 16179_to_12177
- removed joint 16180_to_12177
- removed joint 16181_to_12177
- removed joint 16183_to_12182
- removed joint 16184_to_12182
- removed joint 16185_to_12182
- removed joint 16186_to_12182
- removed joint 1642_to_1241
- removed joint 1643_to_1241
- removed joint 1644_to_1241
- removed joint 1645_to_1241
- removed joint 1647_to_1246
- removed joint 1648_to_1246
- removed joint 1649_to_1246
- removed joint 1650_to_1246
- removed joint 1652_to_1251
- removed joint 1653_to_1251
- removed joint 1654_to_1251
- removed joint 1655_to_1251
- removed joint 1657_to_1256
- removed joint 1658_to_1256
- removed joint 1659_to_1256
- removed joint 1660_to_1256
- removed joint 1667_to_1266
- removed joint 1668_to_1266
- removed joint 1669_to_1266
- removed joint 1670_to_1266
- removed joint 1672_to_1271
- removed joint 1673_to_1271
- removed joint 1674_to_1271
- removed joint 1675_to_1271
- removed joint 1677_to_1276
- removed joint 1678_to_1276
- removed joint 1679_to_1276
- removed joint 1680_to_1276
- removed joint 1682_to_1281
- removed joint 1683_to_1281
- removed joint 1684_to_1281
- removed joint 1685_to_1281
- removed joint 1692_to_1291
- removed joint 1693_to_1291
- removed joint 1694_to_1291
- removed joint 1695_to_1291
- removed joint 1697_to_1296
- removed joint 1698_to_1296
- removed joint 1699_to_1296
- removed joint 1712_to_510
- removed joint 174_to_52
- removed joint 178_to_56
- removed joint 18220_to_0
- removed joint 1917_to_213
- removed joint 1918_to_213
- removed joint 1919_to_213
- removed joint 1920_to_213
- removed joint 1925_to_221
- removed joint 1926_to_221
- removed joint 1927_to_221
- removed joint 1928_to_221
- removed joint 1933_to_229
- removed joint 1934_to_229
- removed joint 1935_to_229
- removed joint 1936_to_229
- removed joint 213_to_0
- removed joint 221_to_0
- removed joint 229_to_0
- removed joint 3113_to_0
- removed joint 337_to_0
- removed joint 4114_to_3113
- removed joint 4139_to_3113
- removed joint 4164_to_3113
- removed joint 438_to_337
- removed joint 463_to_337
- removed joint 488_to_337
- removed joint 510_to_19
- removed joint 52_to_11
- removed joint 56_to_15
- removed joint 6115_to_4114
- removed joint 6116_to_4114
- removed joint 6140_to_4139
- removed joint 6141_to_4139
- removed joint 6165_to_4164
- removed joint 6166_to_4164
- removed joint 639_to_438
- removed joint 640_to_438
- removed joint 664_to_463
- removed joint 665_to_463
- removed joint 689_to_488
- removed joint 690_to_488
- removed joint 7189_to_0
- removed joint 8190_to_7189
- removed joint 8195_to_7189
- removed joint 9200_to_0
- removed joint 9205_to_0
- removed joint 9210_to_0
- removed joint 9215_to_0
- added joint 113_to_0: type revolute, parent 0, child 113, origin xyz=0.588360315768213 0.7144939802055135 0.8759301769331351 rpy=11.97892255531727 3.3803455565831606 3.360197768605905, axis 0 1 0, limit lower=3.1415 upper=-3.1415 effort=1 velocity=1
- added joint 210_to_19: type revolute, parent 19, child 210, origin xyz=0.534221713157885 0.7572050361852153 0.21156947154303396 rpy=11.828824807098005 2.4235413610076293 1.0289950641395593, axis 0 1 0, limit lower=3.1415 upper=-3.1415 effort=1 velocity=1
- added joint 211_to_19: type revolute, parent 19, child 211, origin xyz=0.534221713157885 0.7572050361852153 0.21156947154303396 rpy=17.74323721064701 2.4235413610076293 1.0289950641395593, axis 0 1 0, limit lower=3.1415 upper=-3.1415 effort=1 velocity=1
- added joint 212_to_19: type revolute, parent 19, child 212, origin xyz=0.534221713157885 0.7572050361852153 0.21156947154303396 rpy=23.65764961419601 2.4235413610076293 1.0289950641395593, axis 0 1 0, limit lower=3.1415 upper=-3.1415 effort=1 velocity=1
- added joint 214_to_113: type revolute, parent 113, child 214, origin xyz=0.534221713157885 0.7572050361852153 0.21156947154303396 rpy=11.828824807098005 2.4235413610076293 1.0289950641395593, axis 0 1 0, limit lower=3.1415 upper=-3.1415 effort=1 velocity=1
- added joint 215_to_113: type revolute, parent 113, child 215, origin xyz=0.534221713157885 0.7572050361852153 0.21156947154303396 rpy=17.74323721064701 2.4235413610076293 1.0289950641395593, axis 0 1 0, limit lower=3.1415 upper=-3.1415 effort=1 velocity=1
- added joint 216_to_113: type revolute, parent 113, child 216, origin xyz=0.534221713157885 0.7572050361852153 0.21156947154303396 rpy=23.65764961419601 2.4235413610076293 1.0289950641395593, axis 0 1 0, limit lower=3.1415 upper=-3.1415 effort=1 velocity=1
- added joint 22_to_11: type revolute, parent 11, child 22, origin xyz=0.534221713157885 0.7572050361852153 0.21156947154303396 rpy=11.828824807098005 2.4235413610076293 1.0289950641395593, axis 0 1 0, limit lower=3.1415 upper=-3.1415 effort=1 velocity=1
- added joint 23_to_11: type revolute, parent 11, child 23, origin xyz=0.534221713157885 0.7572050361852153 0.21156947154303396 rpy=17.74323721064701 2.4235413610076293 1.0289950641395593, axis 0 1 0, limit lower=3.1415 upper=-3.1415 effort=1 velocity=1
- added joint 24_to_11: type revolute, parent 11, child 24, origin xyz=0.534221713157885 0.7572050361852153 0.21156947154303396 rpy=23.65764961419601 2.4235413610076293 1.0289950641395593, axis 0 1 0, limit lower=3.1415 upper=-3.1415 effort=1 velocity=1
- added joint 26_to_15: type revolute, parent 15, child 26, origin xyz=0.534221713157885 0.7572050361852153 0.21156947154303396 rpy=11.828824807098005 2.4235413610076293 1.0289950641395593, axis 0 1 0, limit lower=3.1415 upper=-3.1415 effort=1 velocity=1
- added joint 27_to_15: type revolute, parent 15, child 27, origin xyz=0.534221713157885 0.7572050361852153 0.21156947154303396 rpy=17.74323721064701 2.4235413610076293 1.0289950641395593, axis 0 1 0, limit lower=3.1415 upper=-3.1415 effort=1 velocity=1
- added joint 28_to_15: type revolute, parent 15, child 28, origin xyz=0.534221713157885 0.7572050361852153 0.21156947154303396 rpy=23.65764961419601 2.4235413610076293 1.0289950641395593, axis 0 1 0, limit lower=3.1415 upper=-3.1415 effort=1 velocity=1
- joint 11_to_0: origin xyz=0.9674324517982118 0.10812961028432966 0.347652684882915 rpy=0.5411709270436614 1.032004504979393 1.6996450767444733 -> xyz=0.588360315768213 0.7144939802055135 0.8759301769331351 rpy=4.791569022126908 3.3803455565831606 3.360197768605905
- joint 15_to_0: origin xyz=0.9674324517982118 0.10812961028432966 0.347652684882915 rpy=0.8117563905654921 1.032004504979393 1.6996450767444733 -> xyz=0.588360315768213 0.7144939802055135 0.8759301769331351 rpy=7.187353533190363 3.3803455565831606 3.360197768605905
- joint 19_to_0: origin xyz=0.9674324517982118 0.10812961028432966 0.347652684882915 rpy=1.0823418540873229 1.032004504979393 1.6996450767444733 -> xyz=0.588360315768213 0.7144939802055135 0.8759301769331351 rpy=9.583138044253817 3.3803455565831606 3.360197768605905

Commit message: update camera to follow creature

File: test.urdf (robot description, URDF)
Before this commit: robot pepe, 10 links, 9 joints
Joints:
- joint 11_to_0: origin xyz=0.7611592138178738 0.26263827915132143 0.9544215578851041 rpy=11.870000634389736 1.6046171044347293 4.003629441277388 -> xyz=0.8595805157200221 0.26263827915132143 0.9544215578851041 rpy=11.870000634389736 1.6046171044347293 4.003629441277388
- joint 14_to_0: origin xyz=0.7611592138178738 0.26263827915132143 0.9544215578851041 rpy=17.805000951584603 1.6046171044347293 4.003629441277388 -> xyz=0.8595805157200221 0.26263827915132143 0.9544215578851041 rpy=17.805000951584603 1.6046171044347293 4.003629441277388
- joint 17_to_0: origin xyz=0.7611592138178738 0.26263827915132143 0.9544215578851041 rpy=23.740001268779473 1.6046171044347293 4.003629441277388 -> xyz=0.8595805157200221 0.26263827915132143 0.9544215578851041 rpy=23.740001268779473 1.6046171044347293 4.003629441277388
