Commit message: add note to run test_simulation.py outside of ipython

File: temp0.urdf (robot description, URDF)
Before this commit: robot pepe, 6 links, 5 joints
Links:
- link 0: mass 0.04347051203192725 -> 0.056719946520250475; geometry collision cylinder length=0.29153144086541904 radius=0.2488572344229566; visual cylinder length=0.29153144086541904 radius=0.2488572344229566
- link 11: mass 0.005100342146141253 -> 0.4504994334997828; geometry collision cylinder length=0.3098085928862735 radius=0.6803391430326626; visual cylinder length=0.3098085928862735 radius=0.6803391430326626
- link 22: mass 0.4206937501478465 -> 0.06593356131250229; geometry collision cylinder length=0.7842747178728178 radius=0.1635852805552197; visual cylinder length=0.7842747178728178 radius=0.1635852805552197
- link 23: mass 0.4206937501478465 -> 0.06593356131250229; geometry collision cylinder length=0.7842747178728178 radius=0.1635852805552197; visual cylinder length=0.7842747178728178 radius=0.1635852805552197
- link 24: mass 0.4206937501478465 -> 0.06593356131250229; geometry collision cylinder length=0.7842747178728178 radius=0.1635852805552197; visual cylinder length=0.7842747178728178 radius=0.1635852805552197
- link 25: mass 0.4206937501478465 -> 0.06593356131250229; geometry collision cylinder length=0.7842747178728178 radius=0.1635852805552197; visual cylinder length=0.7842747178728178 radius=0.1635852805552197
Joints:
- joint 11_to_0: origin xyz=0.7521023326004612 0.9480186651090544 0.7629739683307908 rpy=5.408803134057071 5.637893656869307 2.729294022443484 -> xyz=0.10150380369073742 0.34432283434548605 0.8216500599510314 rpy=2.3608665297065436 0.2065653201708377 3.012216837926169
- joint 22_to_11: axis 0 1 0 -> 0 0 1; origin xyz=0.08641685938415444 0.6006357600063799 0.3535584227296037 rpy=1.5527121510212911 1.3080765871031113 0.5697859125288693 -> xyz=0.08407356862524229 0.8535470860886838 0.548667642049904 rpy=8.978410336203645 0.44635209542511667 3.8842193279640536
- joint 23_to_11: axis 0 1 0 -> 0 0 1; origin xyz=0.08641685938415444 0.6006357600063799 0.3535584227296037 rpy=2.3290682265319367 1.3080765871031113 0.5697859125288693 -> xyz=0.08407356862524229 0.8535470860886838 0.548667642049904 rpy=13.467615504305467 0.44635209542511667 3.8842193279640536
- joint 24_to_11: axis 0 1 0 -> 0 0 1; origin xyz=0.08641685938415444 0.6006357600063799 0.3535584227296037 rpy=3.1054243020425822 1.3080765871031113 0.5697859125288693 -> xyz=0.08407356862524229 0.8535470860886838 0.548667642049904 rpy=17.95682067240729 0.44635209542511667 3.8842193279640536
- joint 25_to_11: axis 0 1 0 -> 0 0 1; origin xyz=0.08641685938415444 0.6006357600063799 0.3535584227296037 rpy=3.881780377553228 1.3080765871031113 0.5697859125288693 -> xyz=0.08407356862524229 0.8535470860886838 0.548667642049904 rpy=22.44602584050911 0.44635209542511667 3.8842193279640536

File: temp1.urdf (robot description, URDF)
Before this commit: robot pepe, 7 links, 6 joints
Links:
- removed link 23
- added link 13, mass 0.005796148686580906; collision cylinder length=0.17528452880688317 radius=0.10259425207657724; visual cylinder length=0.17528452880688317 radius=0.10259425207657724
- added link 27, mass 0.5644548884602517; collision cylinder length=0.5284323168926627 radius=0.5831026272272751; visual cylinder length=0.5284323168926627 radius=0.5831026272272751
- link 0: mass 1.1386845716600489 -> 2.2853308979250015; geometry collision cylinder length=0.9068003465220729 radius=0.8956612198609273; visual cylinder length=0.9068003465220729 radius=0.8956612198609273
- link 11: mass 1.2324593185984505 -> 0.005796148686580906; geometry collision cylinder length=0.17528452880688317 radius=0.10259425207657724; visual cylinder length=0.17528452880688317 radius=0.10259425207657724
- link 12: mass 1.2324593185984505 -> 0.005796148686580906; geometry collision cylinder length=0.17528452880688317 radius=0.10259425207657724; visual cylinder length=0.17528452880688317 radius=0.10259425207657724
- link 24: mass 0.02987220705500808 -> 0.5644548884602517; geometry collision cylinder length=0.5284323168926627 radius=0.5831026272272751; visual cylinder length=0.5284323168926627 radius=0.5831026272272751
- link 25: mass 0.02987220705500808 -> 0.5644548884602517; geometry collision cylinder length=0.5284323168926627 radius=0.5831026272272751; visual cylinder length=0.5284323168926627 radius=0.5831026272272751
- link 26: mass 0.02987220705500808 -> 0.5644548884602517; geometry collision cylinder length=0.5284323168926627 radius=0.5831026272272751; visual cylinder length=0.5284323168926627 radius=0.5831026272272751
Joints:
- removed joint 23_to_0
- added joint 13_to_0: type revolute, parent 0, child 13, origin xyz=0.5981472401964166 0.6837668493997091 0.3309743206386433 rpy=7.843169551620996 4.579208367830996 1.767410602776518, axis 0 1 0, limit lower=3.1415 upper=-3.1415 effort=1 velocity=1
- added joint 27_to_0: type revolute, parent 0, child 27, origin xyz=0.6243419250113228 0.13848085640355667 0.2909787552741978 rpy=4.1788251086318855 3.2512058550525254 4.063865690242365, axis 0 0 1, limit lower=3.1415 upper=-3.1415 effort=1 velocity=1
- joint 11_to_0: origin xyz=0.014740189953014182 0.5396949134979394 0.030694446853445134 rpy=9.2036356338335 5.362428997896359 1.1493827907658651 -> xyz=0.5981472401964166 0.6837668493997091 0.3309743206386433 rpy=3.921584775810498 4.579208367830996 1.767410602776518
- joint 12_to_0: origin xyz=0.014740189953014182 0.5396949134979394 0.030694446853445134 rpy=13.80545345075025 5.362428997896359 1.1493827907658651 -> xyz=0.5981472401964166 0.6837668493997091 0.3309743206386433 rpy=5.882377163715747 4.579208367830996 1.767410602776518
- joint 24_to_0: axis 1 0 0 -> 0 0 1; origin xyz=0.2430716928715918 0.22903627956807715 0.013737210904421815 rpy=9.350630873643887 3.049565281496748 0.6352422494443691 -> xyz=0.6243419250113228 0.13848085640355667 0.2909787552741978 rpy=2.611765692894928 3.2512058550525254 4.063865690242365
- joint 25_to_0: axis 1 0 0 -> 0 0 1; origin xyz=0.2430716928715918 0.22903627956807715 0.013737210904421815 rpy=11.220757048372665 3.049565281496748 0.6352422494443691 -> xyz=0.6243419250113228 0.13848085640355667 0.2909787552741978 rpy=3.134118831473914 3.2512058550525254 4.063865690242365
- joint 26_to_0: axis 1 0 0 -> 0 0 1; origin xyz=0.2430716928715918 0.22903627956807715 0.013737210904421815 rpy=13.090883223101441 3.049565281496748 0.6352422494443691 -> xyz=0.6243419250113228 0.13848085640355667 0.2909787552741978 rpy=3.6564719700529 3.2512058550525254 4.063865690242365

File: temp2.urdf (robot description, URDF)
Before this commit: robot pepe, 6 links, 5 joints
Links:
- removed link 12
- removed link 14
- removed link 25
- added link 15, mass 0.1160743071039241; collision cylinder length=0.5552255279039253 radius=0.2579635831597812; visual cylinder length=0.5552255279039253 radius=0.2579635831597812
- added link 17, mass 0.1160743071039241; collision cylinder length=0.5552255279039253 radius=0.2579635831597812; visual cylinder length=0.5552255279039253 radius=0.2579635831597812
- added link 22, mass 0.1477415432749106; collision cylinder length=0.9120764048203853 radius=0.22707052751669854; visual cylinder length=0.9120764048203853 radius=0.22707052751669854
- added link 24, mass 0.1477415432749106; collision cylinder length=0.9120764048203853 radius=0.22707052751669854; visual cylinder length=0.9120764048203853 radius=0.22707052751669854
- added link 26, mass 0.1477415432749106; collision cylinder length=0.9120764048203853 radius=0.22707052751669854; visual cylinder length=0.9120764048203853 radius=0.22707052751669854
- added link 28, mass 0.1477415432749106; collision cylinder length=0.9120764048203853 radius=0.22707052751669854; visual cylinder length=0.9120764048203853 radius=0.22707052751669854
- link 0: mass 0.03144547057414081 -> 2.7523101715011373; geometry collision cylinder length=0.9803151556135613 radius=0.9453462217127899; visual cylinder length=0.9803151556135613 radius=0.9453462217127899
- link 11: mass 2.383693103459142 -> 0.1160743071039241; geometry collision cylinder length=0.5552255279039253 radius=0.2579635831597812; visual cylinder length=0.5552255279039253 radius=0.2579635831597812
- link 13: mass 2.383693103459142 -> 0.1160743071039241; geometry collision cylinder length=0.5552255279039253 radius=0.2579635831597812; visual cylinder length=0.5552255279039253 radius=0.2579635831597812
Joints:
- removed joint 12_to_0
- removed joint 14_to_0
- removed joint 25_to_0
- added joint 15_to_0: type revolute, parent 0, child 15, origin xyz=0.6272106166922962 0.21176605765536027 0.4480087464323598 rpy=10.559537547404979 5.33341798195908 2.427282067818647, axis 0 1 0, limit lower=3.1415 upper=-3.1415 effort=1 velocity=1
- added joint 17_to_0: type revolute, parent 0, child 17, origin xyz=0.6272106166922962 0.21176605765536027 0.4480087464323598 rpy=13.199421934256224 5.33341798195908 2.427282067818647, axis 0 1 0, limit lower=3.1415 upper=-3.1415 effort=1 velocity=1
- added joint 22_to_11: type revolute, parent 11, child 22, origin xyz=0.26503680566185417 0.3846730049887397 0.5590504781442388 rpy=0.9792699236951871 1.6693050112776948 0.6478034950528259, axis 0 1 0, limit lower=3.1415 upper=-3.1415 effort=1 velocity=1
- added joint 24_to_13: type revolute, parent 13, child 24, origin xyz=0.26503680566185417 0.3846730049887397 0.5590504781442388 rpy=0.9792699236951871 1.6693050112776948 0.6478034950528259, axis 0 1 0, limit lower=3.1415 upper=-3.1415 effort=1 velocity=1
- added joint 26_to_15: type revolute, parent 15, child 26, origin xyz=0.26503680566185417 0.3846730049887397 0.5590504781442388 rpy=0.9792699236951871 1.6693050112776948 0.6478034950528259, axis 0 1 0, limit lower=3.1415 upper=-3.1415 effort=1 velocity=1
- added joint 28_to_17: type revolute, parent 17, child 28, origin xyz=0.26503680566185417 0.3846730049887397 0.5590504781442388 rpy=0.9792699236951871 1.6693050112776948 0.6478034950528259, axis 0 1 0, limit lower=3.1415 upper=-3.1415 effort=1 velocity=1
- joint 11_to_0: axis 1 0 0 -> 0 1 0; origin xyz=0.06798344377073473 0.5709848052373205 0.9055208301028375 rpy=6.346569207584647 1.934051768701825 1.3179211988635182 -> xyz=0.6272106166922962 0.21176605765536027 0.4480087464323598 rpy=5.279768773702489 5.33341798195908 2.427282067818647
- joint 13_to_0: axis 1 0 0 -> 0 1 0; origin xyz=0.06798344377073473 0.5709848052373205 0.9055208301028375 rpy=12.693138415169294 1.934051768701825 1.3179211988635182 -> xyz=0.6272106166922962 0.21176605765536027 0.4480087464323598 rpy=7.919653160553734 5.33341798195908 2.427282067818647

File: temp3.urdf (robot description, URDF)
Before this commit: robot pepe, 5 links, 4 joints
Links:
- removed link 13
- added link 15, mass 1.6390072666514175; collision cylinder length=0.770830887507494 radius=0.8226894893907053; visual cylinder length=0.770830887507494 radius=0.8226894893907053
- added link 23, mass 0.03867159938222178; collision cylinder length=0.19208061565313428 radius=0.2531508332086072; visual cylinder length=0.19208061565313428 radius=0.2531508332086072
- added link 26, mass 0.03867159938222178; collision cylinder length=0.19208061565313428 radius=0.2531508332086072; visual cylinder length=0.19208061565313428 radius=0.2531508332086072
- added link 27, mass 0.03867159938222178; collision cylinder length=0.19208061565313428 radius=0.2531508332086072; visual cylinder length=0.19208061565313428 radius=0.2531508332086072
- added link 28, mass 0.03867159938222178; collision cylinder length=0.19208061565313428 radius=0.2531508332086072; visual cylinder length=0.19208061565313428 radius=0.2531508332086072
- link 0: mass 0.7029375652139432 -> 0.9694459477196559; geometry collision cylinder length=0.838836912834688 radius=0.6065241485691155; visual cylinder length=0.838836912834688 radius=0.6065241485691155
- link 11: mass 0.006142491051952853 -> 1.6390072666514175; geometry collision cylinder length=0.770830887507494 radius=0.8226894893907053; visual cylinder length=0.770830887507494 radius=0.8226894893907053
- link 22: mass 0.9659871774671127 -> 0.03867159938222178; geometry collision cylinder length=0.19208061565313428 radius=0.2531508332086072; visual cylinder length=0.19208061565313428 radius=0.2531508332086072
- link 24: mass 0.9659871774671127 -> 0.03867159938222178; geometry collision cylinder length=0.19208061565313428 radius=0.2531508332086072; visual cylinder length=0.19208061565313428 radius=0.2531508332086072
Joints:
- removed joint 13_to_0
- removed joint 24_to_13
- added joint 15_to_0: type revolute, parent 0, child 15, origin xyz=0.11735432136907897 0.01201470122286541 0.3395072903966563 rpy=10.829518568829261 5.062294171260698 5.014112013523304, axis 0 1 0, limit lower=3.1415 upper=-3.1415 effort=1 velocity=1
- added joint 23_to_11: type revolute, parent 11, child 23, origin xyz=0.288733310296705 0.00980000302474715 0.9180975492951681 rpy=14.156724673030656 2.844999884663126 4.130016442372747, axis 1 0 0, limit lower=3.1415 upper=-3.1415 effort=1 velocity=1
- added joint 24_to_11: type revolute, parent 11, child 24, origin xyz=0.288733310296705 0.00980000302474715 0.9180975492951681 rpy=18.875632897374206 2.844999884663126 4.130016442372747, axis 1 0 0, limit lower=3.1415 upper=-3.1415 effort=1 velocity=1
- added joint 26_to_15: type revolute, parent 15, child 26, origin xyz=0.288733310296705 0.00980000302474715 0.9180975492951681 rpy=9.437816448687103 2.844999884663126 4.130016442372747, axis 1 0 0, limit lower=3.1415 upper=-3.1415 effort=1 velocity=1
- added joint 27_to_15: type revolute, parent 15, child 27, origin xyz=0.288733310296705 0.00980000302474715 0.9180975492951681 rpy=14.156724673030656 2.844999884663126 4.130016442372747, axis 1 0 0, limit lower=3.1415 upper=-3.1415 effort=1 velocity=1
- added joint 28_to_15: type revolute, parent 15, child 28, origin xyz=0.288733310296705 0.00980000302474715 0.9180975492951681 rpy=18.875632897374206 2.844999884663126 4.130016442372747, axis 1 0 0, limit lower=3.1415 upper=-3.1415 effort=1 velocity=1
- joint 11_to_0: axis 0 0 1 -> 0 1 0; origin xyz=0.13964936821445662 0.9467466802753118 0.5269241652254824 rpy=5.416846263661991 1.8758769314554198 5.756188190019519 -> xyz=0.11735432136907897 0.01201470122286541 0.3395072903966563 rpy=7.219679045886174 5.062294171260698 5.014112013523304
- joint 22_to_11: axis 0 1 0 -> 1 0 0; origin xyz=0.2695820798534396 0.17447192425989322 0.616327942580527 rpy=4.720353367528521 4.089860697198579 5.309253897237312 -> xyz=0.288733310296705 0.00980000302474715 0.9180975492951681 rpy=9.437816448687103 2.844999884663126 4.130016442372747
