Commit message: change distance metric to allow back and forth movement

File: temp0.urdf (robot description, URDF)
Before this commit: robot pepe, 14 links, 13 joints
Links:
- removed link 13
- removed link 29
- removed link 310
- removed link 35
- removed link 411
- removed link 412
- removed link 413
- removed link 46
- removed link 47
- removed link 48
- added link 23, mass 0.009290833977696132; collision cylinder length=0.3820965905006577 radius=0.08797632819885409; visual cylinder length=0.3820965905006577 radius=0.08797632819885409
- added link 25, mass 0.009290833977696132; collision cylinder length=0.3820965905006577 radius=0.08797632819885409; visual cylinder length=0.3820965905006577 radius=0.08797632819885409
- added link 36, mass 1.0542435746390661; collision cylinder length=0.47873618895081393 radius=0.83723507812674; visual cylinder length=0.47873618895081393 radius=0.83723507812674
- added link 37, mass 1.0542435746390661; collision cylinder length=0.47873618895081393 radius=0.83723507812674; visual cylinder length=0.47873618895081393 radius=0.83723507812674
- link 0: mass 0.0064604176374358875 -> 0.0060722298511448605; geometry collision cylinder length=0.016136948851283806 radius=0.3460895240892162; visual cylinder length=0.016136948851283806 radius=0.3460895240892162
- link 11: mass 0.7500050911628182 -> 0.3503882476091541; geometry collision cylinder length=0.18959202448349888 radius=0.7669901686478788; visual cylinder length=0.18959202448349888 radius=0.7669901686478788
- link 12: mass 0.7500050911628182 -> 0.3503882476091541; geometry collision cylinder length=0.18959202448349888 radius=0.7669901686478788; visual cylinder length=0.18959202448349888 radius=0.7669901686478788
- link 24: mass 0.5910518647734716 -> 0.009290833977696132; geometry collision cylinder length=0.3820965905006577 radius=0.08797632819885409; visual cylinder length=0.3820965905006577 radius=0.08797632819885409
Joints:
- removed joint 13_to_0
- removed joint 29_to_0
- removed joint 310_to_29
- removed joint 35_to_24
- removed joint 411_to_310
- removed joint 412_to_310
- removed joint 413_to_310
- removed joint 46_to_35
- removed joint 47_to_35
- removed joint 48_to_35
- added joint 23_to_0: type revolute, parent 0, child 23, origin xyz=0.052269880848787253 0.8061694095075347 0.4089083237316975 rpy=11.044730016460337 4.45914966589873 1.0604263560398164, axis 0 0 1, limit lower=3.1415 upper=-3.1415 effort=1 velocity=1
- added joint 25_to_0: type revolute, parent 0, child 25, origin xyz=0.052269880848787253 0.8061694095075347 0.4089083237316975 rpy=16.567095024690506 4.45914966589873 1.0604263560398164, axis 0 0 1, limit lower=3.1415 upper=-3.1415 effort=1 velocity=1
- added joint 36_to_0: type revolute, parent 0, child 36, origin xyz=0.08567222345446368 0.24299484257419157 0.9831121552511143 rpy=35.75376411287067 2.3763127697311552 6.0317205382454775, axis 0 1 0, limit lower=3.1415 upper=-3.1415 effort=1 velocity=1
- added joint 37_to_0: type revolute, parent 0, child 37, origin xyz=0.08567222345446368 0.24299484257419157 0.9831121552511143 rpy=40.86144470042362 2.3763127697311552 6.0317205382454775, axis 0 1 0, limit lower=3.1415 upper=-3.1415 effort=1 velocity=1
- joint 11_to_0: axis 1 0 0 -> 0 0 1; origin xyz=0.8189271008336009 0.7563699647312384 0.9146125821125136 rpy=10.623475154237155 2.136005126326262 3.1496784475622124 -> xyz=0.15986039852037626 0.89154775402469 0.8579656493726011 rpy=2.8323644764938667 1.293594387544998 2.9678389505507834
- joint 12_to_0: axis 1 0 0 -> 0 0 1; origin xyz=0.8189271008336009 0.7563699647312384 0.9146125821125136 rpy=15.935212731355733 2.136005126326262 3.1496784475622124 -> xyz=0.15986039852037626 0.89154775402469 0.8579656493726011 rpy=4.2485467147408 1.293594387544998 2.9678389505507834
- joint 24_to_0: origin xyz=0.026822661312480456 0.7657070746088926 0.9703833558210094 rpy=8.492888449428452 0.9050096959036379 3.6076154805198013 -> xyz=0.052269880848787253 0.8061694095075347 0.4089083237316975 rpy=13.80591252057542 4.45914966589873 1.0604263560398164

File: temp1.urdf (robot description, URDF)
Before this commit: robot pepe, 18 links, 17 joints
Links:
- removed link 111
- removed link 16
- removed link 216
- removed link 217
- removed link 310
- removed link 312
- removed link 313
- removed link 314
- removed link 315
- removed link 32
- removed link 33
- removed link 34
- removed link 35
- removed link 37
- removed link 38
- removed link 39
- added link 12, mass 0.009290833977696132; collision cylinder length=0.3820965905006577 radius=0.08797632819885409; visual cylinder length=0.3820965905006577 radius=0.08797632819885409
- added link 13, mass 0.009290833977696132; collision cylinder length=0.3820965905006577 radius=0.08797632819885409; visual cylinder length=0.3820965905006577 radius=0.08797632819885409
- link 0: mass 0.0064604176374358875 -> 0.3503882476091541; geometry collision cylinder length=0.18959202448349888 radius=0.7669901686478788; visual cylinder length=0.18959202448349888 radius=0.7669901686478788
- link 11: mass 0.7500050911628182 -> 0.009290833977696132; geometry collision cylinder length=0.3820965905006577 radius=0.08797632819885409; visual cylinder length=0.3820965905006577 radius=0.08797632819885409
Joints:
- removed joint 111_to_0
- removed joint 16_to_0
- removed joint 216_to_0
- removed joint 217_to_0
- removed joint 310_to_16
- removed joint 312_to_111
- removed joint 313_to_111
- removed joint 314_to_111
- removed joint 315_to_111
- removed joint 32_to_11
- removed joint 33_to_11
- removed joint 34_to_11
- removed joint 35_to_11
- removed joint 37_to_16
- removed joint 38_to_16
- removed joint 39_to_16
- added joint 12_to_0: type revolute, parent 0, child 12, origin xyz=0.052269880848787253 0.8061694095075347 0.4089083237316975 rpy=8.283547512345253 4.45914966589873 1.0604263560398164, axis 0 0 1, limit lower=3.1415 upper=-3.1415 effort=1 velocity=1
- added joint 13_to_0: type revolute, parent 0, child 13, origin xyz=0.052269880848787253 0.8061694095075347 0.4089083237316975 rpy=11.044730016460337 4.45914966589873 1.0604263560398164, axis 0 0 1, limit lower=3.1415 upper=-3.1415 effort=1 velocity=1
- joint 11_to_0: axis 1 0 0 -> 0 0 1; origin xyz=0.8189271008336009 0.7563699647312384 0.9146125821125136 rpy=10.623475154237155 2.8342104177696292 3.1496784475622124 -> xyz=0.052269880848787253 0.8061694095075347 0.4089083237316975 rpy=5.522365008230168 4.45914966589873 1.0604263560398164

File: temp2.urdf (robot description, URDF)
Before this commit: robot pepe, 5 links, 4 joints
Links:
- added link 25, mass 0.009290833977696132; collision cylinder length=0.3820965905006577 radius=0.08797632819885409; visual cylinder length=0.3820965905006577 radius=0.08797632819885409
- link 0: mass 0.0064604176374358875 -> 0.008887824201159696; geometry collision cylinder length=0.016136948851283806 radius=0.41870879207200407; visual cylinder length=0.016136948851283806 radius=0.41870879207200407
- link 11: mass 0.06845945895472486 -> 0.3503882476091541; geometry collision cylinder length=0.18959202448349888 radius=0.7669901686478788; visual cylinder length=0.18959202448349888 radius=0.7669901686478788
- link 12: mass 0.06845945895472486 -> 0.3503882476091541; geometry collision cylinder length=0.18959202448349888 radius=0.7669901686478788; visual cylinder length=0.18959202448349888 radius=0.7669901686478788
- link 23: mass 0.5910518647734716 -> 0.009290833977696132; geometry collision cylinder length=0.3820965905006577 radius=0.08797632819885409; visual cylinder length=0.3820965905006577 radius=0.08797632819885409
- link 24: mass 0.5910518647734716 -> 0.009290833977696132; geometry collision cylinder length=0.3820965905006577 radius=0.08797632819885409; visual cylinder length=0.3820965905006577 radius=0.08797632819885409
Joints:
- added joint 25_to_0: type revolute, parent 0, child 25, origin xyz=0.052269880848787253 0.8061694095075347 0.4089083237316975 rpy=16.567095024690506 4.45914966589873 1.0604263560398164, axis 0 0 1, limit lower=3.1415 upper=-3.1415 effort=1 velocity=1
- joint 11_to_0: origin xyz=0.6356337499132794 0.6031902401349394 0.23405451282220213 rpy=9.808126357122962 2.5233665411156254 4.787943064201908 -> xyz=0.15986039852037626 0.89154775402469 0.8579656493726011 rpy=2.8323644764938667 1.293594387544998 2.9678389505507834
- joint 12_to_0: origin xyz=0.6356337499132794 0.6031902401349394 0.23405451282220213 rpy=14.712189535684443 2.5233665411156254 4.787943064201908 -> xyz=0.15986039852037626 0.89154775402469 0.8579656493726011 rpy=4.2485467147408 1.293594387544998 2.9678389505507834
- joint 23_to_0: origin xyz=0.026822661312480456 0.7657070746088926 0.9703833558210094 rpy=6.794310759542762 0.9050096959036379 3.6076154805198013 -> xyz=0.052269880848787253 0.8061694095075347 0.4089083237316975 rpy=11.044730016460337 4.45914966589873 1.0604263560398164
- joint 24_to_0: origin xyz=0.026822661312480456 0.7657070746088926 0.9703833558210094 rpy=8.492888449428452 0.9050096959036379 3.6076154805198013 -> xyz=0.052269880848787253 0.8061694095075347 0.4089083237316975 rpy=13.80591252057542 4.45914966589873 1.0604263560398164

File: temp3.urdf (robot description, URDF)
Before this commit: robot pepe, 23 links, 22 joints
Links:
- removed link 111
- removed link 16
- removed link 216
- removed link 217
- removed link 218
- removed link 219
- removed link 320
- removed link 321
- removed link 322
- removed link 410
- removed link 412
- removed link 413
- removed link 414
- removed link 415
- removed link 42
- removed link 43
- removed link 44
- removed link 45
- removed link 47
- removed link 48
- removed link 49
- added link 12, mass 0.3503882476091541; collision cylinder length=0.18959202448349888 radius=0.7669901686478788; visual cylinder length=0.18959202448349888 radius=0.7669901686478788
- added link 23, mass 0.009290833977696132; collision cylinder length=0.3820965905006577 radius=0.08797632819885409; visual cylinder length=0.3820965905006577 radius=0.08797632819885409
- added link 24, mass 0.009290833977696132; collision cylinder length=0.3820965905006577 radius=0.08797632819885409; visual cylinder length=0.3820965905006577 radius=0.08797632819885409
- added link 25, mass 0.009290833977696132; collision cylinder length=0.3820965905006577 radius=0.08797632819885409; visual cylinder length=0.3820965905006577 radius=0.08797632819885409
- link 0: mass 0.0064604176374358875 -> 0.008887824201159696; geometry collision cylinder length=0.016136948851283806 radius=0.41870879207200407; visual cylinder length=0.016136948851283806 radius=0.41870879207200407
- link 11: mass 0.7500050911628182 -> 0.3503882476091541; geometry collision cylinder length=0.18959202448349888 radius=0.7669901686478788; visual cylinder length=0.18959202448349888 radius=0.7669901686478788
Joints:
- removed joint 111_to_0
- removed joint 16_to_0
- removed joint 216_to_0
- removed joint 217_to_0
- removed joint 218_to_0
- removed joint 219_to_0
- removed joint 320_to_0
- removed joint 321_to_0
- removed joint 322_to_0
- removed joint 410_to_16
- removed joint 412_to_111
- removed joint 413_to_111
- removed joint 414_to_111
- removed joint 415_to_111
- removed joint 42_to_11
- removed joint 43_to_11
- removed joint 44_to_11
- removed joint 45_to_11
- removed joint 47_to_16
- removed joint 48_to_16
- removed joint 49_to_16
- added joint 12_to_0: type revolute, parent 0, child 12, origin xyz=0.15986039852037626 0.89154775402469 0.8579656493726011 rpy=4.2485467147408 1.293594387544998 2.9678389505507834, axis 0 0 1, limit lower=3.1415 upper=-3.1415 effort=1 velocity=1
- added joint 23_to_0: type revolute, parent 0, child 23, origin xyz=0.052269880848787253 0.8061694095075347 0.4089083237316975 rpy=11.044730016460337 4.45914966589873 1.0604263560398164, axis 0 0 1, limit lower=3.1415 upper=-3.1415 effort=1 velocity=1
- added joint 24_to_0: type revolute, parent 0, child 24, origin xyz=0.052269880848787253 0.8061694095075347 0.4089083237316975 rpy=13.80591252057542 4.45914966589873 1.0604263560398164, axis 0 0 1, limit lower=3.1415 upper=-3.1415 effort=1 velocity=1
- added joint 25_to_0: type revolute, parent 0, child 25, origin xyz=0.052269880848787253 0.8061694095075347 0.4089083237316975 rpy=16.567095024690506 4.45914966589873 1.0604263560398164, axis 0 0 1, limit lower=3.1415 upper=-3.1415 effort=1 velocity=1
- joint 11_to_0: axis 1 0 0 -> 0 0 1; origin xyz=0.8189271008336009 0.7563699647312384 0.9146125821125136 rpy=10.623475154237155 2.8342104177696292 3.1496784475622124 -> xyz=0.15986039852037626 0.89154775402469 0.8579656493726011 rpy=2.8323644764938667 1.293594387544998 2.9678389505507834

File: temp4.urdf (robot description, URDF)
Before this commit: robot pepe, 12 links, 11 joints
Links:
- removed link 14
- removed link 17
- removed link 210
- removed link 211
- removed link 32
- removed link 33
- removed link 35
- removed link 36
- removed link 38
- removed link 39
- added link 12, mass 0.009290833977696132; collision cylinder length=0.3820965905006577 radius=0.08797632819885409; visual cylinder length=0.3820965905006577 radius=0.08797632819885409
- added link 13, mass 0.009290833977696132; collision cylinder length=0.3820965905006577 radius=0.08797632819885409; visual cylinder length=0.3820965905006577 radius=0.08797632819885409
- link 0: mass 0.0064604176374358875 -> 0.008887824201159696; geometry collision cylinder length=0.016136948851283806 radius=0.41870879207200407; visual cylinder length=0.016136948851283806 radius=0.41870879207200407
- link 11: mass 0.7500050911628182 -> 0.009290833977696132; geometry collision cylinder length=0.3820965905006577 radius=0.08797632819885409; visual cylinder length=0.3820965905006577 radius=0.08797632819885409
Joints:
- removed joint 14_to_0
- removed joint 17_to_0
- removed joint 210_to_0
- removed joint 211_to_0
- removed joint 32_to_11
- removed joint 33_to_11
- removed joint 35_to_14
- removed joint 36_to_14
- removed joint 38_to_17
- removed joint 39_to_17
- added joint 12_to_0: type revolute, parent 0, child 12, origin xyz=0.052269880848787253 0.8061694095075347 0.4089083237316975 rpy=8.283547512345253 4.45914966589873 1.0604263560398164, axis 0 0 1, limit lower=3.1415 upper=-3.1415 effort=1 velocity=1
- added joint 13_to_0: type revolute, parent 0, child 13, origin xyz=0.052269880848787253 0.8061694095075347 0.4089083237316975 rpy=11.044730016460337 4.45914966589873 1.0604263560398164, axis 0 0 1, limit lower=3.1415 upper=-3.1415 effort=1 velocity=1
- joint 11_to_0: axis 1 0 0 -> 0 0 1; origin xyz=0.8189271008336009 0.7563699647312384 0.9146125821125136 rpy=10.623475154237155 2.8342104177696292 3.1496784475622124 -> xyz=0.052269880848787253 0.8061694095075347 0.4089083237316975 rpy=5.522365008230168 4.45914966589873 1.0604263560398164

File: temp5.urdf (robot description, URDF)
Before this commit: robot pepe, 8 links, 7 joints
Links:
- removed link 13
- removed link 26
- removed link 27
- added link 23, mass 0.009290833977696132; collision cylinder length=0.3820965905006577 radius=0.08797632819885409; visual cylinder length=0.3820965905006577 radius=0.08797632819885409
- link 0: mass 0.0064604176374358875 -> 0.008887824201159696; geometry collision cylinder length=0.016136948851283806 radius=0.41870879207200407; visual cylinder length=0.016136948851283806 radius=0.41870879207200407
- link 11: mass 0.5649325347459758 -> 0.3503882476091541; geometry collision cylinder length=0.18959202448349888 radius=0.7669901686478788; visual cylinder length=0.18959202448349888 radius=0.7669901686478788
- link 12: mass 0.5649325347459758 -> 0.3503882476091541; geometry collision cylinder length=0.18959202448349888 radius=0.7669901686478788; visual cylinder length=0.18959202448349888 radius=0.7669901686478788
- link 24: mass 0.5394855650921216 -> 0.009290833977696132; geometry collision cylinder length=0.3820965905006577 radius=0.08797632819885409; visual cylinder length=0.3820965905006577 radius=0.08797632819885409
- link 25: mass 0.5394855650921216 -> 0.009290833977696132; geometry collision cylinder length=0.3820965905006577 radius=0.08797632819885409; visual cylinder length=0.3820965905006577 radius=0.08797632819885409
Joints:
- removed joint 13_to_0
- removed joint 26_to_0
- removed joint 27_to_0
- added joint 23_to_0: type revolute, parent 0, child 23, origin xyz=0.052269880848787253 0.8061694095075347 0.4089083237316975 rpy=11.044730016460337 4.45914966589873 1.0604263560398164, axis 0 0 1, limit lower=3.1415 upper=-3.1415 effort=1 velocity=1
- joint 11_to_0: axis 1 0 0 -> 0 0 1; origin xyz=0.3118866016961451 0.5661440265582555 0.3863162482295788 rpy=5.597962052795528 4.374845030959743 4.138503952253977 -> xyz=0.15986039852037626 0.89154775402469 0.8579656493726011 rpy=2.8323644764938667 1.293594387544998 2.9678389505507834
- joint 12_to_0: axis 1 0 0 -> 0 0 1; origin xyz=0.3118866016961451 0.5661440265582555 0.3863162482295788 rpy=8.396943079193292 4.374845030959743 4.138503952253977 -> xyz=0.15986039852037626 0.89154775402469 0.8579656493726011 rpy=4.2485467147408 1.293594387544998 2.9678389505507834
- joint 24_to_0: axis 0 1 0 -> 0 0 1; origin xyz=0.9232261393428357 0.7779079037726714 0.631538648594243 rpy=6.587835015834406 1.1555748771549694 1.3105326529696615 -> xyz=0.052269880848787253 0.8061694095075347 0.4089083237316975 rpy=13.80591252057542 4.45914966589873 1.0604263560398164
- joint 25_to_0: axis 0 1 0 -> 0 0 1; origin xyz=0.9232261393428357 0.7779079037726714 0.631538648594243 rpy=7.905402019001286 1.1555748771549694 1.3105326529696615 -> xyz=0.052269880848787253 0.8061694095075347 0.4089083237316975 rpy=16.567095024690506 4.45914966589873 1.0604263560398164

File: temp6.urdf (robot description, URDF)
Before this commit: robot pepe, 29 links, 28 joints
Links:
- removed link 24
- removed link 25
- removed link 26
- removed link 27
- removed link 315
- removed link 322
- removed link 38
- removed link 410
- removed link 411
- removed link 412
- removed link 416
- removed link 417
- removed link 418
- removed link 419
- removed link 423
- removed link 424
- removed link 425
- removed link 426
- removed link 49
- removed link 513
- removed link 514
- removed link 520
- removed link 521
- removed link 527
- removed link 528
- link 0: mass 0.0064604176374358875 -> 0.3503882476091541; geometry collision cylinder length=0.18959202448349888 radius=0.7669901686478788; visual cylinder length=0.18959202448349888 radius=0.7669901686478788
- link 11: mass 0.7500050911628182 -> 0.009290833977696132; geometry collision cylinder length=0.3820965905006577 radius=0.08797632819885409; visual cylinder length=0.3820965905006577 radius=0.08797632819885409
- link 12: mass 0.7500050911628182 -> 0.009290833977696132; geometry collision cylinder length=0.3820965905006577 radius=0.08797632819885409; visual cylinder length=0.3820965905006577 radius=0.08797632819885409
- link 13: mass 0.7500050911628182 -> 0.009290833977696132; geometry collision cylinder length=0.3820965905006577 radius=0.08797632819885409; visual cylinder length=0.3820965905006577 radius=0.08797632819885409
Joints:
- removed joint 24_to_0
- removed joint 25_to_0
- removed joint 26_to_0
- removed joint 27_to_0
- removed joint 315_to_0
- removed joint 322_to_0
- removed joint 38_to_0
- removed joint 410_to_38
- removed joint 411_to_38
- removed joint 412_to_38
- removed joint 416_to_315
- removed joint 417_to_315
- removed joint 418_to_315
- removed joint 419_to_315
- removed joint 423_to_322
- removed joint 424_to_322
- removed joint 425_to_322
- removed joint 426_to_322
- removed joint 49_to_38
- removed joint 513_to_38
- removed joint 514_to_38
- removed joint 520_to_315
- removed joint 521_to_315
- removed joint 527_to_322
- removed joint 528_to_322
- joint 11_to_0: axis 1 0 0 -> 0 0 1; origin xyz=0.8189271008336009 0.7563699647312384 0.9146125821125136 rpy=10.623475154237155 2.8342104177696292 3.1496784475622124 -> xyz=0.052269880848787253 0.8061694095075347 0.4089083237316975 rpy=5.522365008230168 4.45914966589873 1.0604263560398164
- joint 12_to_0: axis 1 0 0 -> 0 0 1; origin xyz=0.8189271008336009 0.7563699647312384 0.9146125821125136 rpy=15.935212731355733 2.8342104177696292 3.1496784475622124 -> xyz=0.052269880848787253 0.8061694095075347 0.4089083237316975 rpy=8.283547512345253 4.45914966589873 1.0604263560398164
- joint 13_to_0: axis 1 0 0 -> 0 0 1; origin xyz=0.8189271008336009 0.7563699647312384 0.9146125821125136 rpy=21.24695030847431 2.8342104177696292 3.1496784475622124 -> xyz=0.052269880848787253 0.8061694095075347 0.4089083237316975 rpy=11.044730016460337 4.45914966589873 1.0604263560398164
