Commit message: change distance metric to allow back and forth movement

File: temp7.urdf (robot description, URDF)
Before this commit: robot pepe, 6 links, 5 joints
Links:
- removed link 13
- added link 23, mass 0.009290833977696132; collision cylinder length=0.3820965905006577 radius=0.08797632819885409; visual cylinder length=0.3820965905006577 radius=0.08797632819885409
- link 0: mass 0.0064604176374358875 -> 0.0060722298511448605; geometry collision cylinder length=0.016136948851283806 radius=0.3460895240892162; visual cylinder length=0.016136948851283806 radius=0.3460895240892162
- link 11: mass 0.7500050911628182 -> 0.3503882476091541; geometry collision cylinder length=0.18959202448349888 radius=0.7669901686478788; visual cylinder length=0.18959202448349888 radius=0.7669901686478788
- link 12: mass 0.7500050911628182 -> 0.3503882476091541; geometry collision cylinder length=0.18959202448349888 radius=0.7669901686478788; visual cylinder length=0.18959202448349888 radius=0.7669901686478788
- link 24: mass 0.5910518647734716 -> 0.009290833977696132; geometry collision cylinder length=0.3820965905006577 radius=0.08797632819885409; visual cylinder length=0.3820965905006577 radius=0.08797632819885409
- link 25: mass 0.5910518647734716 -> 0.009290833977696132; geometry collision cylinder length=0.3820965905006577 radius=0.08797632819885409; visual cylinder length=0.3820965905006577 radius=0.08797632819885409
Joints:
- removed joint 13_to_0
- added joint 23_to_0: type revolute, parent 0, child 23, origin xyz=0.052269880848787253 0.8061694095075347 0.4089083237316975 rpy=11.044730016460337 4.45914966589873 1.0604263560398164, axis 0 0 1, limit lower=3.1415 upper=-3.1415 effort=1 velocity=1
- joint 11_to_0: axis 1 0 0 -> 0 0 1; origin xyz=0.8189271008336009 0.7563699647312384 0.9146125821125136 rpy=10.623475154237155 2.8342104177696292 3.1496784475622124 -> xyz=0.15986039852037626 0.89154775402469 0.8579656493726011 rpy=2.8323644764938667 1.293594387544998 2.9678389505507834
- joint 12_to_0: axis 1 0 0 -> 0 0 1; origin xyz=0.8189271008336009 0.7563699647312384 0.9146125821125136 rpy=15.935212731355733 2.8342104177696292 3.1496784475622124 -> xyz=0.15986039852037626 0.89154775402469 0.8579656493726011 rpy=4.2485467147408 1.293594387544998 2.9678389505507834
- joint 24_to_0: origin xyz=0.026822661312480456 0.7657070746088926 0.9703833558210094 rpy=8.492888449428452 0.9050096959036379 3.6076154805198013 -> xyz=0.052269880848787253 0.8061694095075347 0.4089083237316975 rpy=13.80591252057542 4.45914966589873 1.0604263560398164
- joint 25_to_0: origin xyz=0.026822661312480456 0.7657070746088926 0.9703833558210094 rpy=10.191466139314144 0.9050096959036379 3.6076154805198013 -> xyz=0.052269880848787253 0.8061694095075347 0.4089083237316975 rpy=16.567095024690506 4.45914966589873 1.0604263560398164
