Commit message: implement run_genome.py to see fit creatures

File: temp0.urdf (robot description, URDF)
Before this commit: robot pepe, 8 links, 7 joints
Links:
- removed link 23
- removed link 24
- removed link 25
- removed link 36
- removed link 37
- added link 13, mass 2.6950541517302082; collision cylinder length=0.9724069702602065 radius=0.9392577343978782; visual cylinder length=0.9724069702602065 radius=0.9392577343978782
- link 0: mass 0.0060722298511448605 -> 0.18302461024354932; geometry collision cylinder length=0.2514329775891432 radius=0.4813585494165482; visual cylinder length=0.2514329775891432 radius=0.4813585494165482
- link 11: mass 0.3503882476091541 -> 2.6950541517302082; geometry collision cylinder length=0.9724069702602065 radius=0.9392577343978782; visual cylinder length=0.9724069702602065 radius=0.9392577343978782
- link 12: mass 0.3503882476091541 -> 2.6950541517302082; geometry collision cylinder length=0.9724069702602065 radius=0.9392577343978782; visual cylinder length=0.9724069702602065 radius=0.9392577343978782
Joints:
- removed joint 23_to_0
- removed joint 24_to_0
- removed joint 25_to_0
- removed joint 36_to_0
- removed joint 37_to_0
- added joint 13_to_0: type revolute, parent 0, child 13, origin xyz=0.7611592138178738 0.26263827915132143 0.9544215578851041 rpy=23.740001268779473 1.6046171044347293 4.003629441277388, axis 0 1 0, limit lower=3.1415 upper=-3.1415 effort=1 velocity=1
- joint 11_to_0: axis 0 0 1 -> 0 1 0; origin xyz=0.15986039852037626 0.89154775402469 0.8579656493726011 rpy=2.8323644764938667 1.293594387544998 2.9678389505507834 -> xyz=0.7611592138178738 0.26263827915132143 0.9544215578851041 rpy=11.870000634389736 1.6046171044347293 4.003629441277388
- joint 12_to_0: axis 0 0 1 -> 0 1 0; origin xyz=0.15986039852037626 0.89154775402469 0.8579656493726011 rpy=4.2485467147408 1.293594387544998 2.9678389505507834 -> xyz=0.7611592138178738 0.26263827915132143 0.9544215578851041 rpy=17.805000951584603 1.6046171044347293 4.003629441277388

File: temp1.urdf (robot description, URDF)
Before this commit: robot pepe, 4 links, 3 joints
Links:
- link 0: mass 0.3503882476091541 -> 0.18302461024354932; geometry collision cylinder length=0.2514329775891432 radius=0.4813585494165482; visual cylinder length=0.2514329775891432 radius=0.4813585494165482
- link 11: mass 0.009290833977696132 -> 2.6950541517302082; geometry collision cylinder length=0.9724069702602065 radius=0.9392577343978782; visual cylinder length=0.9724069702602065 radius=0.9392577343978782
- link 12: mass 0.009290833977696132 -> 2.6950541517302082; geometry collision cylinder length=0.9724069702602065 radius=0.9392577343978782; visual cylinder length=0.9724069702602065 radius=0.9392577343978782
- link 13: mass 0.009290833977696132 -> 2.6950541517302082; geometry collision cylinder length=0.9724069702602065 radius=0.9392577343978782; visual cylinder length=0.9724069702602065 radius=0.9392577343978782
Joints:
- joint 11_to_0: axis 0 0 1 -> 0 1 0; origin xyz=0.052269880848787253 0.8061694095075347 0.4089083237316975 rpy=5.522365008230168 4.45914966589873 1.0604263560398164 -> xyz=0.8595805157200221 0.26263827915132143 0.9544215578851041 rpy=11.870000634389736 1.6046171044347293 4.003629441277388
- joint 12_to_0: axis 0 0 1 -> 0 1 0; origin xyz=0.052269880848787253 0.8061694095075347 0.4089083237316975 rpy=8.283547512345253 4.45914966589873 1.0604263560398164 -> xyz=0.8595805157200221 0.26263827915132143 0.9544215578851041 rpy=17.805000951584603 1.6046171044347293 4.003629441277388
- joint 13_to_0: axis 0 0 1 -> 0 1 0; origin xyz=0.052269880848787253 0.8061694095075347 0.4089083237316975 rpy=11.044730016460337 4.45914966589873 1.0604263560398164 -> xyz=0.8595805157200221 0.26263827915132143 0.9544215578851041 rpy=23.740001268779473 1.6046171044347293 4.003629441277388

File: temp2.urdf (robot description, URDF)
Before this commit: robot pepe, 6 links, 5 joints
Links:
- removed link 23
- removed link 24
- removed link 25
- added link 13, mass 2.6950541517302082; collision cylinder length=0.9724069702602065 radius=0.9392577343978782; visual cylinder length=0.9724069702602065 radius=0.9392577343978782
- link 0: mass 0.008887824201159696 -> 0.21443480929550102; geometry collision cylinder length=0.29708679793674075 radius=0.47932604767649856; visual cylinder length=0.29708679793674075 radius=0.47932604767649856
- link 11: mass 0.3503882476091541 -> 2.6950541517302082; geometry collision cylinder length=0.9724069702602065 radius=0.9392577343978782; visual cylinder length=0.9724069702602065 radius=0.9392577343978782
- link 12: mass 0.3503882476091541 -> 2.6950541517302082; geometry collision cylinder length=0.9724069702602065 radius=0.9392577343978782; visual cylinder length=0.9724069702602065 radius=0.9392577343978782
Joints:
- removed joint 23_to_0
- removed joint 24_to_0
- removed joint 25_to_0
- added joint 13_to_0: type revolute, parent 0, child 13, origin xyz=0.7611592138178738 0.26263827915132143 0.9544215578851041 rpy=23.740001268779473 1.6046171044347293 4.003629441277388, axis 0 1 0, limit lower=3.1415 upper=-3.1415 effort=1 velocity=1
- joint 11_to_0: axis 0 0 1 -> 0 1 0; origin xyz=0.15986039852037626 0.89154775402469 0.8579656493726011 rpy=2.8323644764938667 1.293594387544998 2.9678389505507834 -> xyz=0.7611592138178738 0.26263827915132143 0.9544215578851041 rpy=11.870000634389736 1.6046171044347293 4.003629441277388
- joint 12_to_0: axis 0 0 1 -> 0 1 0; origin xyz=0.15986039852037626 0.89154775402469 0.8579656493726011 rpy=4.2485467147408 1.293594387544998 2.9678389505507834 -> xyz=0.7611592138178738 0.26263827915132143 0.9544215578851041 rpy=17.805000951584603 1.6046171044347293 4.003629441277388

File: temp3.urdf (robot description, URDF)
Before this commit: robot pepe, 6 links, 5 joints
Links:
- removed link 12
- removed link 24
- added link 14, mass 2.6950541517302082; collision cylinder length=0.9724069702602065 radius=0.9392577343978782; visual cylinder length=0.9724069702602065 radius=0.9392577343978782
- added link 17, mass 2.6950541517302082; collision cylinder length=0.9724069702602065 radius=0.9392577343978782; visual cylinder length=0.9724069702602065 radius=0.9392577343978782
- added link 22, mass 0.26979691668443595; collision cylinder length=0.8157967461195692 radius=0.32445357987726464; visual cylinder length=0.8157967461195692 radius=0.32445357987726464
- added link 26, mass 0.26979691668443595; collision cylinder length=0.8157967461195692 radius=0.32445357987726464; visual cylinder length=0.8157967461195692 radius=0.32445357987726464
- added link 28, mass 0.26979691668443595; collision cylinder length=0.8157967461195692 radius=0.32445357987726464; visual cylinder length=0.8157967461195692 radius=0.32445357987726464
- added link 29, mass 0.26979691668443595; collision cylinder length=0.8157967461195692 radius=0.32445357987726464; visual cylinder length=0.8157967461195692 radius=0.32445357987726464
- link 0: mass 0.008887824201159696 -> 0.18302461024354932; geometry collision cylinder length=0.2514329775891432 radius=0.4813585494165482; visual cylinder length=0.2514329775891432 radius=0.4813585494165482
- link 11: mass 0.3503882476091541 -> 2.6950541517302082; geometry collision cylinder length=0.9724069702602065 radius=0.9392577343978782; visual cylinder length=0.9724069702602065 radius=0.9392577343978782
- link 23: mass 0.009290833977696132 -> 0.26979691668443595; geometry collision cylinder length=0.8157967461195692 radius=0.32445357987726464; visual cylinder length=0.8157967461195692 radius=0.32445357987726464
- link 25: mass 0.009290833977696132 -> 0.26979691668443595; geometry collision cylinder length=0.8157967461195692 radius=0.32445357987726464; visual cylinder length=0.8157967461195692 radius=0.32445357987726464
Joints:
- removed joint 12_to_0
- removed joint 23_to_0
- removed joint 24_to_0
- removed joint 25_to_0
- added joint 14_to_0: type revolute, parent 0, child 14, origin xyz=0.7611592138178738 0.26263827915132143 0.9544215578851041 rpy=17.805000951584603 1.6046171044347293 4.003629441277388, axis 0 1 0, limit lower=3.1415 upper=-3.1415 effort=1 velocity=1
- added joint 17_to_0: type revolute, parent 0, child 17, origin xyz=0.7611592138178738 0.26263827915132143 0.9544215578851041 rpy=23.740001268779473 1.6046171044347293 4.003629441277388, axis 0 1 0, limit lower=3.1415 upper=-3.1415 effort=1 velocity=1
- added joint 22_to_11: type revolute, parent 11, child 22, origin xyz=0.3018089232343095 0.19770403714540463 0.392045896834455 rpy=4.925507931950128 1.9938912850860744 0.707773777047744, axis 0 0 1, limit lower=3.1415 upper=-3.1415 effort=1 velocity=1
- added joint 23_to_11: type revolute, parent 11, child 23, origin xyz=0.3018089232343095 0.19770403714540463 0.392045896834455 rpy=7.388261897925192 1.9938912850860744 0.707773777047744, axis 0 0 1, limit lower=3.1415 upper=-3.1415 effort=1 velocity=1
- added joint 25_to_14: type revolute, parent 14, child 25, origin xyz=0.3018089232343095 0.19770403714540463 0.392045896834455 rpy=4.925507931950128 1.9938912850860744 0.707773777047744, axis 0 0 1, limit lower=3.1415 upper=-3.1415 effort=1 velocity=1
- added joint 26_to_14: type revolute, parent 14, child 26, origin xyz=0.3018089232343095 0.19770403714540463 0.392045896834455 rpy=7.388261897925192 1.9938912850860744 0.707773777047744, axis 0 0 1, limit lower=3.1415 upper=-3.1415 effort=1 velocity=1
- added joint 28_to_17: type revolute, parent 17, child 28, origin xyz=0.3018089232343095 0.19770403714540463 0.392045896834455 rpy=4.925507931950128 1.9938912850860744 0.707773777047744, axis 0 0 1, limit lower=3.1415 upper=-3.1415 effort=1 velocity=1
- added joint 29_to_17: type revolute, parent 17, child 29, origin xyz=0.3018089232343095 0.19770403714540463 0.392045896834455 rpy=7.388261897925192 1.9938912850860744 0.707773777047744, axis 0 0 1, limit lower=3.1415 upper=-3.1415 effort=1 velocity=1
- joint 11_to_0: axis 0 0 1 -> 0 1 0; origin xyz=0.15986039852037626 0.89154775402469 0.8579656493726011 rpy=2.8323644764938667 1.293594387544998 2.9678389505507834 -> xyz=0.7611592138178738 0.26263827915132143 0.9544215578851041 rpy=11.870000634389736 1.6046171044347293 4.003629441277388

File: temp4.urdf (robot description, URDF)
Before this commit: robot pepe, 4 links, 3 joints
Links:
- removed link 12
- removed link 13
- added link 14, mass 2.6950541517302082; collision cylinder length=0.9724069702602065 radius=0.9392577343978782; visual cylinder length=0.9724069702602065 radius=0.9392577343978782
- added link 17, mass 2.6950541517302082; collision cylinder length=0.9724069702602065 radius=0.9392577343978782; visual cylinder length=0.9724069702602065 radius=0.9392577343978782
- added link 22, mass 0.26979691668443595; collision cylinder length=0.8157967461195692 radius=0.32445357987726464; visual cylinder length=0.8157967461195692 radius=0.32445357987726464
- added link 23, mass 0.26979691668443595; collision cylinder length=0.8157967461195692 radius=0.32445357987726464; visual cylinder length=0.8157967461195692 radius=0.32445357987726464
- added link 25, mass 0.26979691668443595; collision cylinder length=0.8157967461195692 radius=0.32445357987726464; visual cylinder length=0.8157967461195692 radius=0.32445357987726464
- added link 26, mass 0.26979691668443595; collision cylinder length=0.8157967461195692 radius=0.32445357987726464; visual cylinder length=0.8157967461195692 radius=0.32445357987726464
- added link 28, mass 0.26979691668443595; collision cylinder length=0.8157967461195692 radius=0.32445357987726464; visual cylinder length=0.8157967461195692 radius=0.32445357987726464
- added link 29, mass 0.26979691668443595; collision cylinder length=0.8157967461195692 radius=0.32445357987726464; visual cylinder length=0.8157967461195692 radius=0.32445357987726464
- added link 310, mass 0.13863103540233496; collision cylinder length=0.31253496550250237 radius=0.37575605801517764; visual cylinder length=0.31253496550250237 radius=0.37575605801517764
- added link 411, mass 0.09077128782379054; collision cylinder length=0.23960097637949873 radius=0.34726020752561193; visual cylinder length=0.23960097637949873 radius=0.34726020752561193
- added link 412, mass 0.09077128782379054; collision cylinder length=0.23960097637949873 radius=0.34726020752561193; visual cylinder length=0.23960097637949873 radius=0.34726020752561193
- added link 413, mass 0.09077128782379054; collision cylinder length=0.23960097637949873 radius=0.34726020752561193; visual cylinder length=0.23960097637949873 radius=0.34726020752561193
- link 0: mass 0.008887824201159696 -> 0.18302461024354932; geometry collision cylinder length=0.2514329775891432 radius=0.4813585494165482; visual cylinder length=0.2514329775891432 radius=0.4813585494165482
- link 11: mass 0.009290833977696132 -> 2.6950541517302082; geometry collision cylinder length=0.9724069702602065 radius=0.9392577343978782; visual cylinder length=0.9724069702602065 radius=0.9392577343978782
Joints:
- removed joint 12_to_0
- removed joint 13_to_0
- added joint 14_to_0: type revolute, parent 0, child 14, origin xyz=0.8595805157200221 0.26263827915132143 0.9544215578851041 rpy=17.805000951584603 1.6046171044347293 4.003629441277388, axis 0 1 0, limit lower=3.1415 upper=-3.1415 effort=1 velocity=1
- added joint 17_to_0: type revolute, parent 0, child 17, origin xyz=0.8595805157200221 0.26263827915132143 0.9544215578851041 rpy=23.740001268779473 1.6046171044347293 4.003629441277388, axis 0 1 0, limit lower=3.1415 upper=-3.1415 effort=1 velocity=1
- added joint 22_to_11: type revolute, parent 11, child 22, origin xyz=0.3018089232343095 0.19770403714540463 0.392045896834455 rpy=4.925507931950128 1.9938912850860744 0.707773777047744, axis 0 0 1, limit lower=3.1415 upper=-3.1415 effort=1 velocity=1
- added joint 23_to_11: type revolute, parent 11, child 23, origin xyz=0.3018089232343095 0.19770403714540463 0.392045896834455 rpy=7.388261897925192 1.9938912850860744 0.707773777047744, axis 0 0 1, limit lower=3.1415 upper=-3.1415 effort=1 velocity=1
- added joint 25_to_14: type revolute, parent 14, child 25, origin xyz=0.3018089232343095 0.19770403714540463 0.392045896834455 rpy=4.925507931950128 1.9938912850860744 0.707773777047744, axis 0 0 1, limit lower=3.1415 upper=-3.1415 effort=1 velocity=1
- added joint 26_to_14: type revolute, parent 14, child 26, origin xyz=0.3018089232343095 0.19770403714540463 0.392045896834455 rpy=7.388261897925192 1.9938912850860744 0.707773777047744, axis 0 0 1, limit lower=3.1415 upper=-3.1415 effort=1 velocity=1
- added joint 28_to_17: type revolute, parent 17, child 28, origin xyz=0.3018089232343095 0.19770403714540463 0.392045896834455 rpy=4.925507931950128 1.9938912850860744 0.707773777047744, axis 0 0 1, limit lower=3.1415 upper=-3.1415 effort=1 velocity=1
- added joint 29_to_17: type revolute, parent 17, child 29, origin xyz=0.3018089232343095 0.19770403714540463 0.392045896834455 rpy=7.388261897925192 1.9938912850860744 0.707773777047744, axis 0 0 1, limit lower=3.1415 upper=-3.1415 effort=1 velocity=1
- added joint 310_to_0: type revolute, parent 0, child 310, origin xyz=0.26054380147416933 0.6530402882042914 0.16106488141066266 rpy=17.800196041655607 2.7511320262002803 4.750793003916342, axis 1 0 0, limit lower=3.1415 upper=-3.1415 effort=1 velocity=1
- added joint 411_to_0: type revolute, parent 0, child 411, origin xyz=0.3490828221432195 0.4500157532170159 0.4787570525070909 rpy=0.7757331815548862 5.292815221969711 5.46636228827883, axis 1 0 0, limit lower=3.1415 upper=-3.1415 effort=1 velocity=1
- added joint 412_to_0: type revolute, parent 0, child 412, origin xyz=0.3490828221432195 0.4500157532170159 0.4787570525070909 rpy=0.9050220451473673 5.292815221969711 5.46636228827883, axis 1 0 0, limit lower=3.1415 upper=-3.1415 effort=1 velocity=1
- added joint 413_to_0: type revolute, parent 0, child 413, origin xyz=0.3490828221432195 0.4500157532170159 0.4787570525070909 rpy=1.0343109087398483 5.292815221969711 5.46636228827883, axis 1 0 0, limit lower=3.1415 upper=-3.1415 effort=1 velocity=1
- joint 11_to_0: axis 0 0 1 -> 0 1 0; origin xyz=0.052269880848787253 0.8061694095075347 0.4089083237316975 rpy=5.522365008230168 4.45914966589873 1.0604263560398164 -> xyz=0.8595805157200221 0.26263827915132143 0.9544215578851041 rpy=11.870000634389736 1.6046171044347293 4.003629441277388

File: temp6.urdf (robot description, URDF)
Before this commit: robot pepe, 4 links, 3 joints
Links:
- removed link 12
- removed link 13
- added link 14, mass 2.6950541517302082; collision cylinder length=0.9724069702602065 radius=0.9392577343978782; visual cylinder length=0.9724069702602065 radius=0.9392577343978782
- added link 17, mass 2.6950541517302082; collision cylinder length=0.9724069702602065 radius=0.9392577343978782; visual cylinder length=0.9724069702602065 radius=0.9392577343978782
- added link 22, mass 0.26979691668443595; collision cylinder length=0.8157967461195692 radius=0.32445357987726464; visual cylinder length=0.8157967461195692 radius=0.32445357987726464
- added link 23, mass 0.26979691668443595; collision cylinder length=0.8157967461195692 radius=0.32445357987726464; visual cylinder length=0.8157967461195692 radius=0.32445357987726464
- added link 25, mass 0.26979691668443595; collision cylinder length=0.8157967461195692 radius=0.32445357987726464; visual cylinder length=0.8157967461195692 radius=0.32445357987726464
- added link 26, mass 0.26979691668443595; collision cylinder length=0.8157967461195692 radius=0.32445357987726464; visual cylinder length=0.8157967461195692 radius=0.32445357987726464
- added link 28, mass 0.26979691668443595; collision cylinder length=0.8157967461195692 radius=0.32445357987726464; visual cylinder length=0.8157967461195692 radius=0.32445357987726464
- added link 29, mass 0.26979691668443595; collision cylinder length=0.8157967461195692 radius=0.32445357987726464; visual cylinder length=0.8157967461195692 radius=0.32445357987726464
- added link 310, mass 0.02781941313071133; collision cylinder length=0.26264248158970627 radius=0.18361855234033975; visual cylinder length=0.26264248158970627 radius=0.18361855234033975
- added link 311, mass 0.02781941313071133; collision cylinder length=0.26264248158970627 radius=0.18361855234033975; visual cylinder length=0.26264248158970627 radius=0.18361855234033975
- added link 312, mass 0.02781941313071133; collision cylinder length=0.26264248158970627 radius=0.18361855234033975; visual cylinder length=0.26264248158970627 radius=0.18361855234033975
- link 0: mass 0.3503882476091541 -> 0.18302461024354932; geometry collision cylinder length=0.2514329775891432 radius=0.4813585494165482; visual cylinder length=0.2514329775891432 radius=0.4813585494165482
- link 11: mass 0.009290833977696132 -> 2.6950541517302082; geometry collision cylinder length=0.9724069702602065 radius=0.9392577343978782; visual cylinder length=0.9724069702602065 radius=0.9392577343978782
Joints:
- removed joint 12_to_0
- removed joint 13_to_0
- added joint 14_to_0: type revolute, parent 0, child 14, origin xyz=0.7611592138178738 0.26263827915132143 0.9544215578851041 rpy=17.805000951584603 1.6046171044347293 4.003629441277388, axis 0 1 0, limit lower=3.1415 upper=-3.1415 effort=1 velocity=1
- added joint 17_to_0: type revolute, parent 0, child 17, origin xyz=0.7611592138178738 0.26263827915132143 0.9544215578851041 rpy=23.740001268779473 1.6046171044347293 4.003629441277388, axis 0 1 0, limit lower=3.1415 upper=-3.1415 effort=1 velocity=1
- added joint 22_to_11: type revolute, parent 11, child 22, origin xyz=0.3018089232343095 0.19770403714540463 0.392045896834455 rpy=4.925507931950128 1.9938912850860744 0.707773777047744, axis 0 0 1, limit lower=3.1415 upper=-3.1415 effort=1 velocity=1
- added joint 23_to_11: type revolute, parent 11, child 23, origin xyz=0.3018089232343095 0.19770403714540463 0.392045896834455 rpy=7.388261897925192 1.9938912850860744 0.707773777047744, axis 0 0 1, limit lower=3.1415 upper=-3.1415 effort=1 velocity=1
- added joint 25_to_14: type revolute, parent 14, child 25, origin xyz=0.3018089232343095 0.19770403714540463 0.392045896834455 rpy=4.925507931950128 1.9938912850860744 0.707773777047744, axis 0 0 1, limit lower=3.1415 upper=-3.1415 effort=1 velocity=1
- added joint 26_to_14: type revolute, parent 14, child 26, origin xyz=0.3018089232343095 0.19770403714540463 0.392045896834455 rpy=7.388261897925192 1.9938912850860744 0.707773777047744, axis 0 0 1, limit lower=3.1415 upper=-3.1415 effort=1 velocity=1
- added joint 28_to_17: type revolute, parent 17, child 28, origin xyz=0.3018089232343095 0.19770403714540463 0.392045896834455 rpy=4.925507931950128 1.9938912850860744 0.707773777047744, axis 0 0 1, limit lower=3.1415 upper=-3.1415 effort=1 velocity=1
- added joint 29_to_17: type revolute, parent 17, child 29, origin xyz=0.3018089232343095 0.19770403714540463 0.392045896834455 rpy=7.388261897925192 1.9938912850860744 0.707773777047744, axis 0 0 1, limit lower=3.1415 upper=-3.1415 effort=1 velocity=1
- added joint 310_to_0: type revolute, parent 0, child 310, origin xyz=0.12254074350822408 0.3648144969918299 0.17142991860581258 rpy=1.4746569238811085 3.6850640218778414 4.85315252788258, axis 0 1 0, limit lower=3.1415 upper=-3.1415 effort=1 velocity=1
- added joint 311_to_0: type revolute, parent 0, child 311, origin xyz=0.12254074350822408 0.3648144969918299 0.17142991860581258 rpy=1.7695883086573303 3.6850640218778414 4.85315252788258, axis 0 1 0, limit lower=3.1415 upper=-3.1415 effort=1 velocity=1
- added joint 312_to_0: type revolute, parent 0, child 312, origin xyz=0.12254074350822408 0.3648144969918299 0.17142991860581258 rpy=2.064519693433552 3.6850640218778414 4.85315252788258, axis 0 1 0, limit lower=3.1415 upper=-3.1415 effort=1 velocity=1
- joint 11_to_0: axis 0 0 1 -> 0 1 0; origin xyz=0.052269880848787253 0.8061694095075347 0.4089083237316975 rpy=5.522365008230168 4.45914966589873 1.0604263560398164 -> xyz=0.7611592138178738 0.26263827915132143 0.9544215578851041 rpy=11.870000634389736 1.6046171044347293 4.003629441277388
