Commit message: implement run_genome.py to see fit creatures

File: temp7.urdf (robot description, URDF)
Before this commit: robot pepe, 6 links, 5 joints
Links:
- removed link 24
- removed link 25
- added link 34, mass 0.3589541103584202; collision cylinder length=0.2040564871830005 radius=0.7482889396425668; visual cylinder length=0.2040564871830005 radius=0.7482889396425668
- added link 35, mass 0.3589541103584202; collision cylinder length=0.2040564871830005 radius=0.7482889396425668; visual cylinder length=0.2040564871830005 radius=0.7482889396425668
- added link 36, mass 0.3589541103584202; collision cylinder length=0.2040564871830005 radius=0.7482889396425668; visual cylinder length=0.2040564871830005 radius=0.7482889396425668
- added link 37, mass 0.3589541103584202; collision cylinder length=0.2040564871830005 radius=0.7482889396425668; visual cylinder length=0.2040564871830005 radius=0.7482889396425668
- link 0: mass 0.0060722298511448605 -> 2.8161037643810345; geometry collision cylinder length=0.9724069702602065 radius=0.9601196510178068; visual cylinder length=0.9724069702602065 radius=0.9601196510178068
- link 11: mass 0.3503882476091541 -> 0.26979691668443595; geometry collision cylinder length=0.8157967461195692 radius=0.32445357987726464; visual cylinder length=0.8157967461195692 radius=0.32445357987726464
- link 12: mass 0.3503882476091541 -> 0.26979691668443595; geometry collision cylinder length=0.8157967461195692 radius=0.32445357987726464; visual cylinder length=0.8157967461195692 radius=0.32445357987726464
- link 23: mass 0.009290833977696132 -> 0.13863103540233496; geometry collision cylinder length=0.31253496550250237 radius=0.37575605801517764; visual cylinder length=0.31253496550250237 radius=0.37575605801517764
Joints:
- removed joint 24_to_0
- removed joint 25_to_0
- added joint 34_to_0: type revolute, parent 0, child 34, origin xyz=0.5864566203229808 0.13068199545191084 0.2911647455957018 rpy=6.340075218630197 0.07998476401470773 1.996686727448204, axis 0 1 0, limit lower=3.1415 upper=-3.1415 effort=1 velocity=1
- added joint 35_to_0: type revolute, parent 0, child 35, origin xyz=0.5864566203229808 0.13068199545191084 0.2911647455957018 rpy=7.608090262356236 0.07998476401470773 1.996686727448204, axis 0 1 0, limit lower=3.1415 upper=-3.1415 effort=1 velocity=1
- added joint 36_to_0: type revolute, parent 0, child 36, origin xyz=0.5864566203229808 0.13068199545191084 0.2911647455957018 rpy=8.876105306082275 0.07998476401470773 1.996686727448204, axis 0 1 0, limit lower=3.1415 upper=-3.1415 effort=1 velocity=1
- added joint 37_to_0: type revolute, parent 0, child 37, origin xyz=0.5864566203229808 0.13068199545191084 0.2911647455957018 rpy=10.144120349808315 0.07998476401470773 1.996686727448204, axis 0 1 0, limit lower=3.1415 upper=-3.1415 effort=1 velocity=1
- joint 11_to_0: origin xyz=0.15986039852037626 0.89154775402469 0.8579656493726011 rpy=2.8323644764938667 1.293594387544998 2.9678389505507834 -> xyz=0.3018089232343095 0.19770403714540463 0.392045896834455 rpy=4.925507931950128 1.9938912850860744 0.707773777047744
- joint 12_to_0: origin xyz=0.15986039852037626 0.89154775402469 0.8579656493726011 rpy=4.2485467147408 1.293594387544998 2.9678389505507834 -> xyz=0.3018089232343095 0.19770403714540463 0.392045896834455 rpy=7.388261897925192 1.9938912850860744 0.707773777047744
- joint 23_to_0: axis 0 0 1 -> 1 0 0; origin xyz=0.052269880848787253 0.8061694095075347 0.4089083237316975 rpy=11.044730016460337 4.45914966589873 1.0604263560398164 -> xyz=0.26054380147416933 0.6530402882042914 0.16106488141066266 rpy=14.240156833324486 2.7511320262002803 4.750793003916342

File: test.urdf (robot description, URDF)
Before this commit: robot pepe, 55 links, 54 joints
Links:
- removed link 119
- removed link 137
- removed link 220
- removed link 221
- removed link 238
- removed link 239
- removed link 314
- removed link 322
- removed link 327
- removed link 332
- removed link 34
- removed link 340
- removed link 345
- removed link 350
- removed link 39
- removed link 410
- removed link 411
- removed link 412
- removed link 413
- removed link 415
- removed link 416
- removed link 417
- removed link 418
- removed link 423
- removed link 424
- removed link 425
- removed link 426
- removed link 428
- removed link 429
- removed link 430
- removed link 431
- removed link 433
- removed link 434
- removed link 435
- removed link 436
- removed link 441
- removed link 442
- removed link 443
- removed link 444
- removed link 446
- removed link 447
- removed link 448
- removed link 449
- removed link 45
- removed link 451
- removed link 452
- removed link 453
- removed link 454
- removed link 46
- removed link 47
- removed link 48
- added link 14, mass 2.6950541517302082; collision cylinder length=0.9724069702602065 radius=0.9392577343978782; visual cylinder length=0.9724069702602065 radius=0.9392577343978782
- added link 17, mass 2.6950541517302082; collision cylinder length=0.9724069702602065 radius=0.9392577343978782; visual cylinder length=0.9724069702602065 radius=0.9392577343978782
- added link 25, mass 0.26979691668443595; collision cylinder length=0.8157967461195692 radius=0.32445357987726464; visual cylinder length=0.8157967461195692 radius=0.32445357987726464
- added link 26, mass 0.26979691668443595; collision cylinder length=0.8157967461195692 radius=0.32445357987726464; visual cylinder length=0.8157967461195692 radius=0.32445357987726464
- added link 28, mass 0.26979691668443595; collision cylinder length=0.8157967461195692 radius=0.32445357987726464; visual cylinder length=0.8157967461195692 radius=0.32445357987726464
- added link 29, mass 0.26979691668443595; collision cylinder length=0.8157967461195692 radius=0.32445357987726464; visual cylinder length=0.8157967461195692 radius=0.32445357987726464
- link 0: mass 0.45752019238045055 -> 0.18302461024354932; geometry collision cylinder length=0.2514329775891432 radius=0.4813585494165482; visual cylinder length=0.2514329775891432 radius=0.4813585494165482
- link 11: mass 1.9922967795459348 -> 2.6950541517302082; geometry collision cylinder length=0.9724069702602065 radius=0.9392577343978782; visual cylinder length=0.9724069702602065 radius=0.9392577343978782
- link 22: mass 0.2228649377207587 -> 0.26979691668443595; geometry collision cylinder length=0.8157967461195692 radius=0.32445357987726464; visual cylinder length=0.8157967461195692 radius=0.32445357987726464
- link 23: mass 0.2228649377207587 -> 0.26979691668443595; geometry collision cylinder length=0.8157967461195692 radius=0.32445357987726464; visual cylinder length=0.8157967461195692 radius=0.32445357987726464
Joints:
- removed joint 119_to_0
- removed joint 137_to_0
- removed joint 220_to_119
- removed joint 221_to_119
- removed joint 238_to_137
- removed joint 239_to_137
- removed joint 314_to_11
- removed joint 322_to_119
- removed joint 327_to_119
- removed joint 332_to_119
- removed joint 340_to_137
- removed joint 345_to_137
- removed joint 34_to_11
- removed joint 350_to_137
- removed joint 39_to_11
- removed joint 410_to_39
- removed joint 411_to_39
- removed joint 412_to_39
- removed joint 413_to_39
- removed joint 415_to_314
- removed joint 416_to_314
- removed joint 417_to_314
- removed joint 418_to_314
- removed joint 423_to_322
- removed joint 424_to_322
- removed joint 425_to_322
- removed joint 426_to_322
- removed joint 428_to_327
- removed joint 429_to_327
- removed joint 430_to_327
- removed joint 431_to_327
- removed joint 433_to_332
- removed joint 434_to_332
- removed joint 435_to_332
- removed joint 436_to_332
- removed joint 441_to_340
- removed joint 442_to_340
- removed joint 443_to_340
- removed joint 444_to_340
- removed joint 446_to_345
- removed joint 447_to_345
- removed joint 448_to_345
- removed joint 449_to_345
- removed joint 451_to_350
- removed joint 452_to_350
- removed joint 453_to_350
- removed joint 454_to_350
- removed joint 45_to_34
- removed joint 46_to_34
- removed joint 47_to_34
- removed joint 48_to_34
- added joint 14_to_0: type revolute, parent 0, child 14, origin xyz=0.7611592138178738 0.26263827915132143 0.9544215578851041 rpy=17.805000951584603 1.6046171044347293 4.003629441277388, axis 0 1 0, limit lower=3.1415 upper=-3.1415 effort=1 velocity=1
- added joint 17_to_0: type revolute, parent 0, child 17, origin xyz=0.7611592138178738 0.26263827915132143 0.9544215578851041 rpy=23.740001268779473 1.6046171044347293 4.003629441277388, axis 0 1 0, limit lower=3.1415 upper=-3.1415 effort=1 velocity=1
- added joint 25_to_14: type revolute, parent 14, child 25, origin xyz=0.3018089232343095 0.19770403714540463 0.392045896834455 rpy=4.925507931950128 1.9938912850860744 0.707773777047744, axis 0 0 1, limit lower=3.1415 upper=-3.1415 effort=1 velocity=1
- added joint 26_to_14: type revolute, parent 14, child 26, origin xyz=0.3018089232343095 0.19770403714540463 0.392045896834455 rpy=7.388261897925192 1.9938912850860744 0.707773777047744, axis 0 0 1, limit lower=3.1415 upper=-3.1415 effort=1 velocity=1
- added joint 28_to_17: type revolute, parent 17, child 28, origin xyz=0.3018089232343095 0.19770403714540463 0.392045896834455 rpy=4.925507931950128 1.9938912850860744 0.707773777047744, axis 0 0 1, limit lower=3.1415 upper=-3.1415 effort=1 velocity=1
- added joint 29_to_17: type revolute, parent 17, child 29, origin xyz=0.3018089232343095 0.19770403714540463 0.392045896834455 rpy=7.388261897925192 1.9938912850860744 0.707773777047744, axis 0 0 1, limit lower=3.1415 upper=-3.1415 effort=1 velocity=1
- joint 11_to_0: axis 0 0 1 -> 0 1 0; origin xyz=0.35362981115640146 0.8849129081775543 0.08372428731370674 rpy=11.255027139398504 5.166318824637535 0.6942491317139261 -> xyz=0.7611592138178738 0.26263827915132143 0.9544215578851041 rpy=11.870000634389736 1.6046171044347293 4.003629441277388
- joint 22_to_11: origin xyz=0.3221595825928266 0.7552748145158681 0.294799539339191 rpy=1.812321266055931 3.8199719505239744 3.5480404510740544 -> xyz=0.3018089232343095 0.19770403714540463 0.392045896834455 rpy=4.925507931950128 1.9938912850860744 0.707773777047744
- joint 23_to_11: origin xyz=0.3221595825928266 0.7552748145158681 0.294799539339191 rpy=2.7184818990838964 3.8199719505239744 3.5480404510740544 -> xyz=0.3018089232343095 0.19770403714540463 0.392045896834455 rpy=7.388261897925192 1.9938912850860744 0.707773777047744
