Commit message: make some changes to genetic variation

File: temp0.urdf (robot description, URDF)
Before this commit: robot pepe, 4 links, 3 joints
Links:
- removed link 12
- removed link 13
- added link 24, mass 0.002781356233409099; collision cylinder length=0.6495471760136006 radius=0.03691883791518524; visual cylinder length=0.6495471760136006 radius=0.03691883791518524
- added link 25, mass 0.002781356233409099; collision cylinder length=0.6495471760136006 radius=0.03691883791518524; visual cylinder length=0.6495471760136006 radius=0.03691883791518524
- added link 32, mass 0.706934280521354; collision cylinder length=0.28044304140720944 radius=0.8957612070219065; visual cylinder length=0.28044304140720944 radius=0.8957612070219065
- added link 33, mass 0.706934280521354; collision cylinder length=0.28044304140720944 radius=0.8957612070219065; visual cylinder length=0.28044304140720944 radius=0.8957612070219065
- link 0: mass 0.18302461024354932 -> 0.0656625499606453; geometry collision cylinder length=0.3163732279676421 radius=0.2570301519389081; visual cylinder length=0.3163732279676421 radius=0.2570301519389081
- link 11: mass 2.6950541517302082 -> 0.43893179769285917; geometry collision cylinder length=0.46262696654027 radius=0.5495511403814227; visual cylinder length=0.46262696654027 radius=0.5495511403814227
Joints:
- removed joint 12_to_0
- removed joint 13_to_0
- added joint 24_to_0: type revolute, parent 0, child 24, origin xyz=0.14757575492045916 0.22648433133033752 0.768252755509006 rpy=18.137710816954197 3.5840032023859494 2.00410165214818, axis 1 0 0, limit lower=3.1415 upper=-3.1415 effort=1 velocity=1
- added joint 25_to_0: type revolute, parent 0, child 25, origin xyz=0.14757575492045916 0.22648433133033752 0.768252755509006 rpy=24.183614422605594 3.5840032023859494 2.00410165214818, axis 1 0 0, limit lower=3.1415 upper=-3.1415 effort=1 velocity=1
- added joint 32_to_11: type revolute, parent 11, child 32, origin xyz=0.13188039176825306 0.8711005140798695 0.16146780040063902 rpy=0.9138747879007154 3.283036796296135 3.1515061237507913, axis 0 0 1, limit lower=3.1415 upper=-3.1415 effort=1 velocity=1
- added joint 33_to_11: type revolute, parent 11, child 33, origin xyz=0.13188039176825306 0.8711005140798695 0.16146780040063902 rpy=1.3708121818510732 3.283036796296135 3.1515061237507913, axis 0 0 1, limit lower=3.1415 upper=-3.1415 effort=1 velocity=1
- joint 11_to_0: axis 0 1 0 -> 0 0 1; origin xyz=0.7611592138178738 0.26263827915132143 0.9544215578851041 rpy=11.870000634389736 1.6046171044347293 4.003629441277388 -> xyz=0.8317592498885846 0.6506740518234515 0.08033703312692048 rpy=4.242709261096144 6.242736811171016 1.6189296120094512

File: temp1.urdf (robot description, URDF)
Before this commit: robot pepe, 4 links, 3 joints
Links:
- removed link 12
- removed link 13
- added link 22, mass 0.357073931956523; collision cylinder length=0.7281569920312759 radius=0.3950859853782801; visual cylinder length=0.7281569920312759 radius=0.3950859853782801
- added link 23, mass 0.357073931956523; collision cylinder length=0.7281569920312759 radius=0.3950859853782801; visual cylinder length=0.7281569920312759 radius=0.3950859853782801
- link 0: mass 0.18302461024354932 -> 0.0656625499606453; geometry collision cylinder length=0.3163732279676421 radius=0.2570301519389081; visual cylinder length=0.3163732279676421 radius=0.2570301519389081
- link 11: mass 2.6950541517302082 -> 0.09777328110326605; geometry collision cylinder length=0.09441289300432174 radius=0.574142248387529; visual cylinder length=0.09441289300432174 radius=0.574142248387529
Joints:
- removed joint 12_to_0
- removed joint 13_to_0
- added joint 22_to_11: type revolute, parent 11, child 22, origin xyz=0.4629956474248542 0.15295891958123453 0.2787447681945542 rpy=3.187399433171077 3.1556927090780684 0.22993842633188863, axis 0 1 0, limit lower=3.1415 upper=-3.1415 effort=1 velocity=1
- added joint 23_to_11: type revolute, parent 11, child 23, origin xyz=0.4629956474248542 0.15295891958123453 0.2787447681945542 rpy=4.781099149756615 3.1556927090780684 0.22993842633188863, axis 0 1 0, limit lower=3.1415 upper=-3.1415 effort=1 velocity=1
- joint 11_to_0: axis 0 1 0 -> 1 0 0; origin xyz=0.8595805157200221 0.26263827915132143 0.9544215578851041 rpy=11.870000634389736 1.6046171044347293 4.003629441277388 -> xyz=0.6952506915179402 0.8815945829934303 0.4522187053142819 rpy=6.021208138471891 3.827880140251571 3.497393685292438

File: temp2.urdf (robot description, URDF)
Before this commit: robot pepe, 4 links, 3 joints
Links:
- removed link 12
- removed link 13
- added link 22, mass 0.6762555372256879; collision cylinder length=0.7390980158932943 radius=0.539671473785115; visual cylinder length=0.7390980158932943 radius=0.539671473785115
- added link 23, mass 0.6762555372256879; collision cylinder length=0.7390980158932943 radius=0.539671473785115; visual cylinder length=0.7390980158932943 radius=0.539671473785115
- added link 24, mass 0.6762555372256879; collision cylinder length=0.7390980158932943 radius=0.539671473785115; visual cylinder length=0.7390980158932943 radius=0.539671473785115
- added link 25, mass 0.6762555372256879; collision cylinder length=0.7390980158932943 radius=0.539671473785115; visual cylinder length=0.7390980158932943 radius=0.539671473785115
- added link 36, mass 0.3693130136257478; collision cylinder length=0.3378902440409972 radius=0.5898404375557437; visual cylinder length=0.3378902440409972 radius=0.5898404375557437
- added link 37, mass 0.3693130136257478; collision cylinder length=0.3378902440409972 radius=0.5898404375557437; visual cylinder length=0.3378902440409972 radius=0.5898404375557437
- link 0: mass 0.21443480929550102 -> 0.05272695044460802; geometry collision cylinder length=0.2200615809877765 radius=0.2761654064408394; visual cylinder length=0.2200615809877765 radius=0.2761654064408394
- link 11: mass 2.6950541517302082 -> 0.43893179769285917; geometry collision cylinder length=0.46262696654027 radius=0.5495511403814227; visual cylinder length=0.46262696654027 radius=0.5495511403814227
Joints:
- removed joint 12_to_0
- removed joint 13_to_0
- added joint 22_to_11: type revolute, parent 11, child 22, origin xyz=0.7713827438134189 0.8471844793559141 0.7733132300909366 rpy=1.1685017951966374 2.607990398758587 5.279593793770392, axis 0 0 1, limit lower=3.1415 upper=-3.1415 effort=1 velocity=1
- added joint 23_to_11: type revolute, parent 11, child 23, origin xyz=0.7713827438134189 0.8471844793559141 0.7733132300909366 rpy=1.7527526927949562 2.607990398758587 5.279593793770392, axis 0 0 1, limit lower=3.1415 upper=-3.1415 effort=1 velocity=1
- added joint 24_to_11: type revolute, parent 11, child 24, origin xyz=0.7713827438134189 0.8471844793559141 0.7733132300909366 rpy=2.337003590393275 2.607990398758587 5.279593793770392, axis 0 0 1, limit lower=3.1415 upper=-3.1415 effort=1 velocity=1
- added joint 25_to_11: type revolute, parent 11, child 25, origin xyz=0.7713827438134189 0.8471844793559141 0.7733132300909366 rpy=2.9212544879915936 2.607990398758587 5.279593793770392, axis 0 0 1, limit lower=3.1415 upper=-3.1415 effort=1 velocity=1
- added joint 36_to_0: type revolute, parent 0, child 36, origin xyz=0.3564701274709101 0.7731346677060382 0.5835350714842641 rpy=10.023161449708818 5.071470531415218 3.1593269496086744, axis 0 0 1, limit lower=3.1415 upper=-3.1415 effort=1 velocity=1
- added joint 37_to_0: type revolute, parent 0, child 37, origin xyz=0.3564701274709101 0.7731346677060382 0.5835350714842641 rpy=13.364215266278423 5.071470531415218 3.1593269496086744, axis 0 0 1, limit lower=3.1415 upper=-3.1415 effort=1 velocity=1
- joint 11_to_0: axis 0 1 0 -> 0 0 1; origin xyz=0.7611592138178738 0.26263827915132143 0.9544215578851041 rpy=11.870000634389736 1.6046171044347293 4.003629441277388 -> xyz=0.8317592498885846 0.6506740518234515 0.028898558806017098 rpy=4.242709261096144 6.242736811171016 1.6189296120094512

File: temp3.urdf (robot description, URDF)
Before this commit: robot pepe, 10 links, 9 joints
Links:
- removed link 14
- removed link 17
- removed link 22
- removed link 23
- removed link 25
- removed link 26
- removed link 28
- removed link 29
- link 0: mass 0.18302461024354932 -> 0.0656625499606453; geometry collision cylinder length=0.3163732279676421 radius=0.2570301519389081; visual cylinder length=0.3163732279676421 radius=0.2570301519389081
- link 11: mass 2.6950541517302082 -> 0.09777328110326605; geometry collision cylinder length=0.09441289300432174 radius=0.574142248387529; visual cylinder length=0.09441289300432174 radius=0.574142248387529
Joints:
- removed joint 14_to_0
- removed joint 17_to_0
- removed joint 22_to_11
- removed joint 23_to_11
- removed joint 25_to_14
- removed joint 26_to_14
- removed joint 28_to_17
- removed joint 29_to_17
- joint 11_to_0: axis 0 1 0 -> 1 0 0; origin xyz=0.7611592138178738 0.26263827915132143 0.9544215578851041 rpy=11.870000634389736 1.6046171044347293 4.003629441277388 -> xyz=0.6952506915179402 0.8815945829934303 0.4522187053142819 rpy=6.021208138471891 3.827880140251571 3.497393685292438

File: temp4.urdf (robot description, URDF)
Before this commit: robot pepe, 14 links, 13 joints
Links:
- removed link 14
- removed link 17
- removed link 25
- removed link 26
- removed link 28
- removed link 29
- removed link 310
- removed link 411
- removed link 412
- removed link 413
- added link 34, mass 0.11194192580395648; collision cylinder length=0.11504802571435624 radius=0.5565213955545212; visual cylinder length=0.11504802571435624 radius=0.5565213955545212
- added link 35, mass 0.11194192580395648; collision cylinder length=0.11504802571435624 radius=0.5565213955545212; visual cylinder length=0.11504802571435624 radius=0.5565213955545212
- added link 36, mass 0.11194192580395648; collision cylinder length=0.11504802571435624 radius=0.5565213955545212; visual cylinder length=0.11504802571435624 radius=0.5565213955545212
- added link 37, mass 0.11194192580395648; collision cylinder length=0.11504802571435624 radius=0.5565213955545212; visual cylinder length=0.11504802571435624 radius=0.5565213955545212
- link 0: mass 0.18302461024354932 -> 0.0656625499606453; geometry collision cylinder length=0.3163732279676421 radius=0.2570301519389081; visual cylinder length=0.3163732279676421 radius=0.2570301519389081
- link 11: mass 2.6950541517302082 -> 0.09777328110326605; geometry collision cylinder length=0.09441289300432174 radius=0.574142248387529; visual cylinder length=0.09441289300432174 radius=0.574142248387529
- link 22: mass 0.26979691668443595 -> 0.357073931956523; geometry collision cylinder length=0.7281569920312759 radius=0.3950859853782801; visual cylinder length=0.7281569920312759 radius=0.3950859853782801
- link 23: mass 0.26979691668443595 -> 0.357073931956523; geometry collision cylinder length=0.7281569920312759 radius=0.3950859853782801; visual cylinder length=0.7281569920312759 radius=0.3950859853782801
Joints:
- removed joint 14_to_0
- removed joint 17_to_0
- removed joint 25_to_14
- removed joint 26_to_14
- removed joint 28_to_17
- removed joint 29_to_17
- removed joint 310_to_0
- removed joint 411_to_0
- removed joint 412_to_0
- removed joint 413_to_0
- added joint 34_to_11: type revolute, parent 11, child 34, origin xyz=0.4359458141653988 0.6113559670815871 0.5889783493681191 rpy=14.157449600206828 0.23021835810255625 1.9643530952785648, axis 0 0 1, limit lower=3.1415 upper=-3.1415 effort=1 velocity=1
- added joint 35_to_11: type revolute, parent 11, child 35, origin xyz=0.4359458141653988 0.6113559670815871 0.5889783493681191 rpy=17.696812000258536 0.23021835810255625 1.9643530952785648, axis 0 0 1, limit lower=3.1415 upper=-3.1415 effort=1 velocity=1
- added joint 36_to_11: type revolute, parent 11, child 36, origin xyz=0.4359458141653988 0.6113559670815871 0.5889783493681191 rpy=21.23617440031024 0.23021835810255625 1.9643530952785648, axis 0 0 1, limit lower=3.1415 upper=-3.1415 effort=1 velocity=1
- added joint 37_to_11: type revolute, parent 11, child 37, origin xyz=0.4359458141653988 0.6113559670815871 0.5889783493681191 rpy=24.775536800361948 0.23021835810255625 1.9643530952785648, axis 0 0 1, limit lower=3.1415 upper=-3.1415 effort=1 velocity=1
- joint 11_to_0: axis 0 1 0 -> 1 0 0; origin xyz=0.8595805157200221 0.26263827915132143 0.9544215578851041 rpy=11.870000634389736 1.6046171044347293 4.003629441277388 -> xyz=0.6952506915179402 0.8815945829934303 0.4522187053142819 rpy=6.021208138471891 3.827880140251571 3.497393685292438
- joint 22_to_11: axis 0 0 1 -> 0 1 0; origin xyz=0.3018089232343095 0.19770403714540463 0.392045896834455 rpy=4.925507931950128 1.9938912850860744 0.707773777047744 -> xyz=0.4629956474248542 0.15295891958123453 0.2787447681945542 rpy=3.187399433171077 3.1556927090780684 0.22993842633188863
- joint 23_to_11: axis 0 0 1 -> 0 1 0; origin xyz=0.3018089232343095 0.19770403714540463 0.392045896834455 rpy=7.388261897925192 1.9938912850860744 0.707773777047744 -> xyz=0.4629956474248542 0.15295891958123453 0.2787447681945542 rpy=4.781099149756615 3.1556927090780684 0.22993842633188863

File: temp5.urdf (robot description, URDF)
Before this commit: robot pepe, 10 links, 9 joints
Links:
- removed link 14
- removed link 17
- removed link 22
- removed link 23
- removed link 25
- removed link 26
- removed link 28
- removed link 29
- link 0: mass 0.18302461024354932 -> 0.05272695044460802; geometry collision cylinder length=0.2200615809877765 radius=0.2761654064408394; visual cylinder length=0.2200615809877765 radius=0.2761654064408394
- link 11: mass 2.6950541517302082 -> 0.43893179769285917; geometry collision cylinder length=0.46262696654027 radius=0.5495511403814227; visual cylinder length=0.46262696654027 radius=0.5495511403814227
Joints:
- removed joint 14_to_0
- removed joint 17_to_0
- removed joint 22_to_11
- removed joint 23_to_11
- removed joint 25_to_14
- removed joint 26_to_14
- removed joint 28_to_17
- removed joint 29_to_17
- joint 11_to_0: axis 0 1 0 -> 0 0 1; origin xyz=0.7611592138178738 0.26263827915132143 0.9544215578851041 rpy=11.870000634389736 1.6046171044347293 4.003629441277388 -> xyz=0.8317592498885846 0.6506740518234515 0.028898558806017098 rpy=4.242709261096144 6.242736811171016 1.6189296120094512

File: temp6.urdf (robot description, URDF)
Before this commit: robot pepe, 13 links, 12 joints
Links:
- removed link 310
- removed link 311
- removed link 312
- added link 110, mass 0.6762555372256879; collision cylinder length=0.7390980158932943 radius=0.539671473785115; visual cylinder length=0.7390980158932943 radius=0.539671473785115
- added link 211, mass 0.0848987674694995; collision cylinder length=0.4871520967295079 radius=0.2355285011149646; visual cylinder length=0.4871520967295079 radius=0.2355285011149646
- added link 212, mass 0.0848987674694995; collision cylinder length=0.4871520967295079 radius=0.2355285011149646; visual cylinder length=0.4871520967295079 radius=0.2355285011149646
- link 0: mass 0.18302461024354932 -> 0.05272695044460802; geometry collision cylinder length=0.2200615809877765 radius=0.2761654064408394; visual cylinder length=0.2200615809877765 radius=0.2761654064408394
- link 11: mass 2.6950541517302082 -> 0.6762555372256879; geometry collision cylinder length=0.7390980158932943 radius=0.539671473785115; visual cylinder length=0.7390980158932943 radius=0.539671473785115
- link 14: mass 2.6950541517302082 -> 0.6762555372256879; geometry collision cylinder length=0.7390980158932943 radius=0.539671473785115; visual cylinder length=0.7390980158932943 radius=0.539671473785115
- link 17: mass 2.6950541517302082 -> 0.6762555372256879; geometry collision cylinder length=0.7390980158932943 radius=0.539671473785115; visual cylinder length=0.7390980158932943 radius=0.539671473785115
- link 22: mass 0.26979691668443595 -> 0.0848987674694995; geometry collision cylinder length=0.4871520967295079 radius=0.2355285011149646; visual cylinder length=0.4871520967295079 radius=0.2355285011149646
- link 23: mass 0.26979691668443595 -> 0.0848987674694995; geometry collision cylinder length=0.4871520967295079 radius=0.2355285011149646; visual cylinder length=0.4871520967295079 radius=0.2355285011149646
- link 25: mass 0.26979691668443595 -> 0.0848987674694995; geometry collision cylinder length=0.4871520967295079 radius=0.2355285011149646; visual cylinder length=0.4871520967295079 radius=0.2355285011149646
- link 26: mass 0.26979691668443595 -> 0.0848987674694995; geometry collision cylinder length=0.4871520967295079 radius=0.2355285011149646; visual cylinder length=0.4871520967295079 radius=0.2355285011149646
- link 28: mass 0.26979691668443595 -> 0.0848987674694995; geometry collision cylinder length=0.4871520967295079 radius=0.2355285011149646; visual cylinder length=0.4871520967295079 radius=0.2355285011149646
- link 29: mass 0.26979691668443595 -> 0.0848987674694995; geometry collision cylinder length=0.4871520967295079 radius=0.2355285011149646; visual cylinder length=0.4871520967295079 radius=0.2355285011149646
Joints:
- removed joint 310_to_0
- removed joint 311_to_0
- removed joint 312_to_0
- added joint 110_to_0: type revolute, parent 0, child 110, origin xyz=0.7713827438134189 0.8471844793559141 0.7733132300909366 rpy=2.9212544879915936 2.607990398758587 5.279593793770392, axis 0 0 1, limit lower=3.1415 upper=-3.1415 effort=1 velocity=1
- added joint 211_to_110: type revolute, parent 110, child 211, origin xyz=0.2185246845322868 0.7707014948884033 0.15637817477119464 rpy=11.62505959161293 0.22062271482782447 5.6968441093664515, axis 0 0 1, limit lower=3.1415 upper=-3.1415 effort=1 velocity=1
- added joint 212_to_110: type revolute, parent 110, child 212, origin xyz=0.2185246845322868 0.7707014948884033 0.15637817477119464 rpy=17.437589387419393 0.22062271482782447 5.6968441093664515, axis 0 0 1, limit lower=3.1415 upper=-3.1415 effort=1 velocity=1
- joint 11_to_0: axis 0 1 0 -> 0 0 1; origin xyz=0.7611592138178738 0.26263827915132143 0.9544215578851041 rpy=11.870000634389736 1.6046171044347293 4.003629441277388 -> xyz=0.7713827438134189 0.8471844793559141 0.7733132300909366 rpy=1.1685017951966374 2.607990398758587 5.279593793770392
- joint 14_to_0: axis 0 1 0 -> 0 0 1; origin xyz=0.7611592138178738 0.26263827915132143 0.9544215578851041 rpy=17.805000951584603 1.6046171044347293 4.003629441277388 -> xyz=0.7713827438134189 0.8471844793559141 0.7733132300909366 rpy=1.7527526927949562 2.607990398758587 5.279593793770392
- joint 17_to_0: axis 0 1 0 -> 0 0 1; origin xyz=0.7611592138178738 0.26263827915132143 0.9544215578851041 rpy=23.740001268779473 1.6046171044347293 4.003629441277388 -> xyz=0.7713827438134189 0.8471844793559141 0.7733132300909366 rpy=2.337003590393275 2.607990398758587 5.279593793770392
- joint 22_to_11: origin xyz=0.3018089232343095 0.19770403714540463 0.392045896834455 rpy=4.925507931950128 1.9938912850860744 0.707773777047744 -> xyz=0.2185246845322868 0.7707014948884033 0.15637817477119464 rpy=11.62505959161293 0.22062271482782447 5.6968441093664515
- joint 23_to_11: origin xyz=0.3018089232343095 0.19770403714540463 0.392045896834455 rpy=7.388261897925192 1.9938912850860744 0.707773777047744 -> xyz=0.2185246845322868 0.7707014948884033 0.15637817477119464 rpy=17.437589387419393 0.22062271482782447 5.6968441093664515
- joint 25_to_14: origin xyz=0.3018089232343095 0.19770403714540463 0.392045896834455 rpy=4.925507931950128 1.9938912850860744 0.707773777047744 -> xyz=0.2185246845322868 0.7707014948884033 0.15637817477119464 rpy=11.62505959161293 0.22062271482782447 5.6968441093664515
- joint 26_to_14: origin xyz=0.3018089232343095 0.19770403714540463 0.392045896834455 rpy=7.388261897925192 1.9938912850860744 0.707773777047744 -> xyz=0.2185246845322868 0.7707014948884033 0.15637817477119464 rpy=17.437589387419393 0.22062271482782447 5.6968441093664515
- joint 28_to_17: origin xyz=0.3018089232343095 0.19770403714540463 0.392045896834455 rpy=4.925507931950128 1.9938912850860744 0.707773777047744 -> xyz=0.2185246845322868 0.7707014948884033 0.15637817477119464 rpy=11.62505959161293 0.22062271482782447 5.6968441093664515
- joint 29_to_17: origin xyz=0.3018089232343095 0.19770403714540463 0.392045896834455 rpy=7.388261897925192 1.9938912850860744 0.707773777047744 -> xyz=0.2185246845322868 0.7707014948884033 0.15637817477119464 rpy=17.437589387419393 0.22062271482782447 5.6968441093664515
