Commit message: make some changes to genetic variation

File: temp7.urdf (robot description, URDF)
Before this commit: robot pepe, 8 links, 7 joints
Links:
- removed link 12
- added link 22, mass 0.357073931956523; collision cylinder length=0.7281569920312759 radius=0.3950859853782801; visual cylinder length=0.7281569920312759 radius=0.3950859853782801
- link 0: mass 2.8161037643810345 -> 0.05272695044460802; geometry collision cylinder length=0.2200615809877765 radius=0.2761654064408394; visual cylinder length=0.2200615809877765 radius=0.2761654064408394
- link 11: mass 0.26979691668443595 -> 0.09777328110326605; geometry collision cylinder length=0.09441289300432174 radius=0.574142248387529; visual cylinder length=0.09441289300432174 radius=0.574142248387529
- link 23: mass 0.13863103540233496 -> 0.357073931956523; geometry collision cylinder length=0.7281569920312759 radius=0.3950859853782801; visual cylinder length=0.7281569920312759 radius=0.3950859853782801
- link 34: mass 0.3589541103584202 -> 0.7163755093457327; geometry collision cylinder length=0.47951994034806267 radius=0.6895918069534182; visual cylinder length=0.47951994034806267 radius=0.6895918069534182
- link 35: mass 0.3589541103584202 -> 0.7163755093457327; geometry collision cylinder length=0.47951994034806267 radius=0.6895918069534182; visual cylinder length=0.47951994034806267 radius=0.6895918069534182
- link 36: mass 0.3589541103584202 -> 0.7163755093457327; geometry collision cylinder length=0.47951994034806267 radius=0.6895918069534182; visual cylinder length=0.47951994034806267 radius=0.6895918069534182
- link 37: mass 0.3589541103584202 -> 0.7163755093457327; geometry collision cylinder length=0.47951994034806267 radius=0.6895918069534182; visual cylinder length=0.47951994034806267 radius=0.6895918069534182
Joints:
- removed joint 12_to_0
- removed joint 23_to_0
- added joint 22_to_11: type revolute, parent 11, child 22, origin xyz=0.4629956474248542 0.15295891958123453 0.2787447681945542 rpy=3.187399433171077 3.1556927090780684 0.22993842633188863, axis 0 1 0, limit lower=3.1415 upper=-3.1415 effort=1 velocity=1
- added joint 23_to_11: type revolute, parent 11, child 23, origin xyz=0.4629956474248542 0.15295891958123453 0.2787447681945542 rpy=4.781099149756615 3.1556927090780684 0.22993842633188863, axis 0 1 0, limit lower=3.1415 upper=-3.1415 effort=1 velocity=1
- joint 11_to_0: axis 0 0 1 -> 1 0 0; origin xyz=0.3018089232343095 0.19770403714540463 0.392045896834455 rpy=4.925507931950128 1.9938912850860744 0.707773777047744 -> xyz=0.6952506915179402 0.8815945829934303 0.4522187053142819 rpy=6.021208138471891 3.827880140251571 3.497393685292438
- joint 34_to_0: origin xyz=0.5864566203229808 0.13068199545191084 0.2911647455957018 rpy=6.340075218630197 0.07998476401470773 1.996686727448204 -> xyz=0.3114385233267407 0.9989547181490429 0.6698865323524993 rpy=16.250893405026222 4.6988404271039945 2.0586300526749057
- joint 35_to_0: origin xyz=0.5864566203229808 0.13068199545191084 0.2911647455957018 rpy=7.608090262356236 0.07998476401470773 1.996686727448204 -> xyz=0.3114385233267407 0.9989547181490429 0.6698865323524993 rpy=21.667857873368295 4.6988404271039945 2.0586300526749057
- joint 36_to_0: origin xyz=0.5864566203229808 0.13068199545191084 0.2911647455957018 rpy=8.876105306082275 0.07998476401470773 1.996686727448204 -> xyz=0.3114385233267407 0.9989547181490429 0.6698865323524993 rpy=27.084822341710368 4.6988404271039945 2.0586300526749057
- joint 37_to_0: origin xyz=0.5864566203229808 0.13068199545191084 0.2911647455957018 rpy=10.144120349808315 0.07998476401470773 1.996686727448204 -> xyz=0.3114385233267407 0.9989547181490429 0.6698865323524993 rpy=32.501786810052444 4.6988404271039945 2.0586300526749057

File: test.urdf (robot description, URDF)
Before this commit: robot pepe, 10 links, 9 joints
Links:
- removed link 14
- removed link 17
- removed link 25
- removed link 26
- removed link 28
- removed link 29
- link 0: mass 0.18302461024354932 -> 0.0656625499606453; geometry collision cylinder length=0.3163732279676421 radius=0.2570301519389081; visual cylinder length=0.3163732279676421 radius=0.2570301519389081
- link 11: mass 2.6950541517302082 -> 0.09777328110326605; geometry collision cylinder length=0.09441289300432174 radius=0.574142248387529; visual cylinder length=0.09441289300432174 radius=0.574142248387529
- link 22: mass 0.26979691668443595 -> 0.357073931956523; geometry collision cylinder length=0.7281569920312759 radius=0.3950859853782801; visual cylinder length=0.7281569920312759 radius=0.3950859853782801
- link 23: mass 0.26979691668443595 -> 0.357073931956523; geometry collision cylinder length=0.7281569920312759 radius=0.3950859853782801; visual cylinder length=0.7281569920312759 radius=0.3950859853782801
Joints:
- removed joint 14_to_0
- removed joint 17_to_0
- removed joint 25_to_14
- removed joint 26_to_14
- removed joint 28_to_17
- removed joint 29_to_17
- joint 11_to_0: axis 0 1 0 -> 1 0 0; origin xyz=0.8595805157200221 0.26263827915132143 0.9544215578851041 rpy=11.870000634389736 1.6046171044347293 4.003629441277388 -> xyz=0.6952506915179402 0.8815945829934303 0.4522187053142819 rpy=6.021208138471891 3.827880140251571 3.497393685292438
- joint 22_to_11: axis 0 0 1 -> 0 1 0; origin xyz=0.3018089232343095 0.19770403714540463 0.392045896834455 rpy=4.925507931950128 1.9938912850860744 0.707773777047744 -> xyz=0.4629956474248542 0.15295891958123453 0.2787447681945542 rpy=3.187399433171077 3.1556927090780684 0.22993842633188863
- joint 23_to_11: axis 0 0 1 -> 0 1 0; origin xyz=0.3018089232343095 0.19770403714540463 0.392045896834455 rpy=7.388261897925192 1.9938912850860744 0.707773777047744 -> xyz=0.4629956474248542 0.15295891958123453 0.2787447681945542 rpy=4.781099149756615 3.1556927090780684 0.22993842633188863
