Commit message: update write to csv based on worksheet

File: temp0.urdf (robot description, URDF)
Before this commit: robot pepe, 6 links, 5 joints
Links:
- removed link 32
- removed link 33
- added link 22, mass 1.1078865586730096; collision cylinder length=0.5885490024600376 radius=0.774072067857943; visual cylinder length=0.5885490024600376 radius=0.774072067857943
- added link 23, mass 1.1078865586730096; collision cylinder length=0.5885490024600376 radius=0.774072067857943; visual cylinder length=0.5885490024600376 radius=0.774072067857943
- link 0: mass 0.0656625499606453 -> 0.013079437091548709; geometry collision cylinder length=0.35940935990721423 radius=0.10762790799951505; visual cylinder length=0.35940935990721423 radius=0.10762790799951505
- link 11: mass 0.43893179769285917 -> 0.000346565382932485; geometry collision cylinder length=0.00014309724393646306 radius=0.878015169482812; visual cylinder length=0.00014309724393646306 radius=0.878015169482812
- link 24: mass 0.002781356233409099 -> 1.1078865586730096; geometry collision cylinder length=0.5885490024600376 radius=0.774072067857943; visual cylinder length=0.5885490024600376 radius=0.774072067857943
- link 25: mass 0.002781356233409099 -> 1.1078865586730096; geometry collision cylinder length=0.5885490024600376 radius=0.774072067857943; visual cylinder length=0.5885490024600376 radius=0.774072067857943
Joints:
- removed joint 24_to_0
- removed joint 25_to_0
- removed joint 32_to_11
- removed joint 33_to_11
- added joint 22_to_11: type revolute, parent 11, child 22, origin xyz=0.7174258218115571 0.9241630040425354 0.6345313651243545 rpy=3.187479884946322 0.5826987100304208 1.9187399681391597, axis 0 0 1, limit lower=3.1415 upper=-3.1415 effort=1 velocity=1
- added joint 23_to_11: type revolute, parent 11, child 23, origin xyz=0.7174258218115571 0.9241630040425354 0.6345313651243545 rpy=4.781219827419483 0.5826987100304208 1.9187399681391597, axis 0 0 1, limit lower=3.1415 upper=-3.1415 effort=1 velocity=1
- added joint 24_to_11: type revolute, parent 11, child 24, origin xyz=0.7174258218115571 0.9241630040425354 0.6345313651243545 rpy=6.374959769892644 0.5826987100304208 1.9187399681391597, axis 0 0 1, limit lower=3.1415 upper=-3.1415 effort=1 velocity=1
- added joint 25_to_11: type revolute, parent 11, child 25, origin xyz=0.7174258218115571 0.9241630040425354 0.6345313651243545 rpy=7.968699712365805 0.5826987100304208 1.9187399681391597, axis 0 0 1, limit lower=3.1415 upper=-3.1415 effort=1 velocity=1
- joint 11_to_0: axis 0 0 1 -> 1 0 0; origin xyz=0.8317592498885846 0.6506740518234515 0.08033703312692048 rpy=4.242709261096144 6.242736811171016 1.6189296120094512 -> xyz=0.14857603399565733 0.850922854525532 0.8784038689011624 rpy=0.14649725603420974 4.846653697982699 5.321823417325937

File: temp1.urdf (robot description, URDF)
Before this commit: robot pepe, 4 links, 3 joints
Links:
- added link 24, mass 1.1078865586730096; collision cylinder length=0.5885490024600376 radius=0.774072067857943; visual cylinder length=0.5885490024600376 radius=0.774072067857943
- added link 25, mass 1.1078865586730096; collision cylinder length=0.5885490024600376 radius=0.774072067857943; visual cylinder length=0.5885490024600376 radius=0.774072067857943
- added link 36, mass 0.08656216894796107; collision cylinder length=0.6698241132036055 radius=0.20281904790217475; visual cylinder length=0.6698241132036055 radius=0.20281904790217475
- added link 37, mass 0.08656216894796107; collision cylinder length=0.6698241132036055 radius=0.20281904790217475; visual cylinder length=0.6698241132036055 radius=0.20281904790217475
- added link 38, mass 0.08656216894796107; collision cylinder length=0.6698241132036055 radius=0.20281904790217475; visual cylinder length=0.6698241132036055 radius=0.20281904790217475
- added link 39, mass 0.08656216894796107; collision cylinder length=0.6698241132036055 radius=0.20281904790217475; visual cylinder length=0.6698241132036055 radius=0.20281904790217475
- link 0: mass 0.0656625499606453 -> 0.013079437091548709; geometry collision cylinder length=0.35940935990721423 radius=0.10762790799951505; visual cylinder length=0.35940935990721423 radius=0.10762790799951505
- link 11: mass 0.09777328110326605 -> 0.000346565382932485; geometry collision cylinder length=0.00014309724393646306 radius=0.878015169482812; visual cylinder length=0.00014309724393646306 radius=0.878015169482812
- link 22: mass 0.357073931956523 -> 1.1078865586730096; geometry collision cylinder length=0.5885490024600376 radius=0.774072067857943; visual cylinder length=0.5885490024600376 radius=0.774072067857943
- link 23: mass 0.357073931956523 -> 1.1078865586730096; geometry collision cylinder length=0.5885490024600376 radius=0.774072067857943; visual cylinder length=0.5885490024600376 radius=0.774072067857943
Joints:
- added joint 24_to_11: type revolute, parent 11, child 24, origin xyz=0.7174258218115571 0.9241630040425354 0.6345313651243545 rpy=6.374959769892644 0.5826987100304208 1.9187399681391597, axis 0 0 1, limit lower=3.1415 upper=-3.1415 effort=1 velocity=1
- added joint 25_to_11: type revolute, parent 11, child 25, origin xyz=0.7174258218115571 0.9241630040425354 0.6345313651243545 rpy=7.968699712365805 0.5826987100304208 1.9187399681391597, axis 0 0 1, limit lower=3.1415 upper=-3.1415 effort=1 velocity=1
- added joint 36_to_11: type revolute, parent 11, child 36, origin xyz=0.6462597085189629 0.8247703460954684 0.3225897180783439 rpy=2.2336799387969823 2.753265867417977 0.13256535444230305, axis 0 0 1, limit lower=3.1415 upper=-3.1415 effort=1 velocity=1
- added joint 37_to_11: type revolute, parent 11, child 37, origin xyz=0.6462597085189629 0.8247703460954684 0.3225897180783439 rpy=2.605959928596479 2.753265867417977 0.13256535444230305, axis 0 0 1, limit lower=3.1415 upper=-3.1415 effort=1 velocity=1
- added joint 38_to_11: type revolute, parent 11, child 38, origin xyz=0.6462597085189629 0.8247703460954684 0.3225897180783439 rpy=2.9782399183959765 2.753265867417977 0.13256535444230305, axis 0 0 1, limit lower=3.1415 upper=-3.1415 effort=1 velocity=1
- added joint 39_to_11: type revolute, parent 11, child 39, origin xyz=0.6462597085189629 0.8247703460954684 0.3225897180783439 rpy=3.3505199081954737 2.753265867417977 0.13256535444230305, axis 0 0 1, limit lower=3.1415 upper=-3.1415 effort=1 velocity=1
- joint 11_to_0: origin xyz=0.6952506915179402 0.8815945829934303 0.4522187053142819 rpy=6.021208138471891 3.827880140251571 3.497393685292438 -> xyz=0.14857603399565733 0.850922854525532 0.8784038689011624 rpy=0.14649725603420974 4.846653697982699 5.321823417325937
- joint 22_to_11: axis 0 1 0 -> 0 0 1; origin xyz=0.4629956474248542 0.15295891958123453 0.2787447681945542 rpy=3.187399433171077 3.1556927090780684 0.22993842633188863 -> xyz=0.7174258218115571 0.9241630040425354 0.6345313651243545 rpy=3.187479884946322 0.5826987100304208 1.9187399681391597
- joint 23_to_11: axis 0 1 0 -> 0 0 1; origin xyz=0.4629956474248542 0.15295891958123453 0.2787447681945542 rpy=4.781099149756615 3.1556927090780684 0.22993842633188863 -> xyz=0.7174258218115571 0.9241630040425354 0.6345313651243545 rpy=4.781219827419483 0.5826987100304208 1.9187399681391597

File: temp2.urdf (robot description, URDF)
Before this commit: robot pepe, 8 links, 7 joints
Links:
- removed link 23
- removed link 24
- removed link 25
- removed link 36
- added link 210, mass 0.08656216894796107; collision cylinder length=0.6698241132036055 radius=0.20281904790217475; visual cylinder length=0.6698241132036055 radius=0.20281904790217475
- added link 214, mass 0.08656216894796107; collision cylinder length=0.6698241132036055 radius=0.20281904790217475; visual cylinder length=0.6698241132036055 radius=0.20281904790217475
- added link 26, mass 0.08656216894796107; collision cylinder length=0.6698241132036055 radius=0.20281904790217475; visual cylinder length=0.6698241132036055 radius=0.20281904790217475
- added link 311, mass 1.3010028094564627; collision cylinder length=0.6594143880653701 radius=0.7924739066722428; visual cylinder length=0.6594143880653701 radius=0.7924739066722428
- added link 312, mass 1.3010028094564627; collision cylinder length=0.6594143880653701 radius=0.7924739066722428; visual cylinder length=0.6594143880653701 radius=0.7924739066722428
- added link 313, mass 1.3010028094564627; collision cylinder length=0.6594143880653701 radius=0.7924739066722428; visual cylinder length=0.6594143880653701 radius=0.7924739066722428
- added link 315, mass 1.3010028094564627; collision cylinder length=0.6594143880653701 radius=0.7924739066722428; visual cylinder length=0.6594143880653701 radius=0.7924739066722428
- added link 316, mass 1.3010028094564627; collision cylinder length=0.6594143880653701 radius=0.7924739066722428; visual cylinder length=0.6594143880653701 radius=0.7924739066722428
- added link 317, mass 1.3010028094564627; collision cylinder length=0.6594143880653701 radius=0.7924739066722428; visual cylinder length=0.6594143880653701 radius=0.7924739066722428
- added link 33, mass 1.3010028094564627; collision cylinder length=0.6594143880653701 radius=0.7924739066722428; visual cylinder length=0.6594143880653701 radius=0.7924739066722428
- added link 34, mass 1.3010028094564627; collision cylinder length=0.6594143880653701 radius=0.7924739066722428; visual cylinder length=0.6594143880653701 radius=0.7924739066722428
- added link 35, mass 1.3010028094564627; collision cylinder length=0.6594143880653701 radius=0.7924739066722428; visual cylinder length=0.6594143880653701 radius=0.7924739066722428
- added link 38, mass 1.3010028094564627; collision cylinder length=0.6594143880653701 radius=0.7924739066722428; visual cylinder length=0.6594143880653701 radius=0.7924739066722428
- added link 39, mass 1.3010028094564627; collision cylinder length=0.6594143880653701 radius=0.7924739066722428; visual cylinder length=0.6594143880653701 radius=0.7924739066722428
- link 0: mass 0.05272695044460802 -> 0.013079437091548709; geometry collision cylinder length=0.35940935990721423 radius=0.10762790799951505; visual cylinder length=0.35940935990721423 radius=0.10762790799951505
- link 11: mass 0.43893179769285917 -> 0.000346565382932485; geometry collision cylinder length=0.00014309724393646306 radius=0.878015169482812; visual cylinder length=0.00014309724393646306 radius=0.878015169482812
- link 22: mass 0.6762555372256879 -> 0.08656216894796107; geometry collision cylinder length=0.6698241132036055 radius=0.20281904790217475; visual cylinder length=0.6698241132036055 radius=0.20281904790217475
- link 37: mass 0.3693130136257478 -> 1.3010028094564627; geometry collision cylinder length=0.6594143880653701 radius=0.7924739066722428; visual cylinder length=0.6594143880653701 radius=0.7924739066722428
Joints:
- removed joint 23_to_11
- removed joint 24_to_11
- removed joint 25_to_11
- removed joint 36_to_0
- removed joint 37_to_0
- added joint 210_to_11: type revolute, parent 11, child 210, origin xyz=0.6462597085189629 0.8247703460954684 0.3225897180783439 rpy=1.4891199591979882 2.753265867417977 0.13256535444230305, axis 0 0 1, limit lower=3.1415 upper=-3.1415 effort=1 velocity=1
- added joint 214_to_11: type revolute, parent 11, child 214, origin xyz=0.6462597085189629 0.8247703460954684 0.3225897180783439 rpy=1.8613999489974853 2.753265867417977 0.13256535444230305, axis 0 0 1, limit lower=3.1415 upper=-3.1415 effort=1 velocity=1
- added joint 26_to_11: type revolute, parent 11, child 26, origin xyz=0.6462597085189629 0.8247703460954684 0.3225897180783439 rpy=1.1168399693984912 2.753265867417977 0.13256535444230305, axis 0 0 1, limit lower=3.1415 upper=-3.1415 effort=1 velocity=1
- added joint 311_to_210: type revolute, parent 210, child 311, origin xyz=0.21244740337731205 0.30963795507434566 0.7532611592364375 rpy=5.69284500720614 6.231285609868876 1.6356365506562816, axis 0 0 1, limit lower=3.1415 upper=-3.1415 effort=1 velocity=1
- added joint 312_to_210: type revolute, parent 210, child 312, origin xyz=0.21244740337731205 0.30963795507434566 0.7532611592364375 rpy=8.53926751080921 6.231285609868876 1.6356365506562816, axis 0 0 1, limit lower=3.1415 upper=-3.1415 effort=1 velocity=1
- added joint 313_to_210: type revolute, parent 210, child 313, origin xyz=0.21244740337731205 0.30963795507434566 0.7532611592364375 rpy=11.38569001441228 6.231285609868876 1.6356365506562816, axis 0 0 1, limit lower=3.1415 upper=-3.1415 effort=1 velocity=1
- added joint 315_to_214: type revolute, parent 214, child 315, origin xyz=0.21244740337731205 0.30963795507434566 0.7532611592364375 rpy=5.69284500720614 6.231285609868876 1.6356365506562816, axis 0 0 1, limit lower=3.1415 upper=-3.1415 effort=1 velocity=1
- added joint 316_to_214: type revolute, parent 214, child 316, origin xyz=0.21244740337731205 0.30963795507434566 0.7532611592364375 rpy=8.53926751080921 6.231285609868876 1.6356365506562816, axis 0 0 1, limit lower=3.1415 upper=-3.1415 effort=1 velocity=1
- added joint 317_to_214: type revolute, parent 214, child 317, origin xyz=0.21244740337731205 0.30963795507434566 0.7532611592364375 rpy=11.38569001441228 6.231285609868876 1.6356365506562816, axis 0 0 1, limit lower=3.1415 upper=-3.1415 effort=1 velocity=1
- added joint 33_to_22: type revolute, parent 22, child 33, origin xyz=0.21244740337731205 0.30963795507434566 0.7532611592364375 rpy=5.69284500720614 6.231285609868876 1.6356365506562816, axis 0 0 1, limit lower=3.1415 upper=-3.1415 effort=1 velocity=1
- added joint 34_to_22: type revolute, parent 22, child 34, origin xyz=0.21244740337731205 0.30963795507434566 0.7532611592364375 rpy=8.53926751080921 6.231285609868876 1.6356365506562816, axis 0 0 1, limit lower=3.1415 upper=-3.1415 effort=1 velocity=1
- added joint 35_to_22: type revolute, parent 22, child 35, origin xyz=0.21244740337731205 0.30963795507434566 0.7532611592364375 rpy=11.38569001441228 6.231285609868876 1.6356365506562816, axis 0 0 1, limit lower=3.1415 upper=-3.1415 effort=1 velocity=1
- added joint 37_to_26: type revolute, parent 26, child 37, origin xyz=0.21244740337731205 0.30963795507434566 0.7532611592364375 rpy=5.69284500720614 6.231285609868876 1.6356365506562816, axis 0 0 1, limit lower=3.1415 upper=-3.1415 effort=1 velocity=1
- added joint 38_to_26: type revolute, parent 26, child 38, origin xyz=0.21244740337731205 0.30963795507434566 0.7532611592364375 rpy=8.53926751080921 6.231285609868876 1.6356365506562816, axis 0 0 1, limit lower=3.1415 upper=-3.1415 effort=1 velocity=1
- added joint 39_to_26: type revolute, parent 26, child 39, origin xyz=0.21244740337731205 0.30963795507434566 0.7532611592364375 rpy=11.38569001441228 6.231285609868876 1.6356365506562816, axis 0 0 1, limit lower=3.1415 upper=-3.1415 effort=1 velocity=1
- joint 11_to_0: axis 0 0 1 -> 1 0 0; origin xyz=0.8317592498885846 0.6506740518234515 0.028898558806017098 rpy=4.242709261096144 6.242736811171016 1.6189296120094512 -> xyz=0.14857603399565733 0.850922854525532 0.8784038689011624 rpy=0.14649725603420974 4.846653697982699 5.321823417325937
- joint 22_to_11: origin xyz=0.7713827438134189 0.8471844793559141 0.7733132300909366 rpy=1.1685017951966374 2.607990398758587 5.279593793770392 -> xyz=0.6462597085189629 0.8247703460954684 0.3225897180783439 rpy=0.7445599795989941 2.753265867417977 0.13256535444230305

File: temp3.urdf (robot description, URDF)
Before this commit: robot pepe, 2 links, 1 joints
Links:
- added link 22, mass 1.1078865586730096; collision cylinder length=0.5885490024600376 radius=0.774072067857943; visual cylinder length=0.5885490024600376 radius=0.774072067857943
- added link 23, mass 1.1078865586730096; collision cylinder length=0.5885490024600376 radius=0.774072067857943; visual cylinder length=0.5885490024600376 radius=0.774072067857943
- added link 24, mass 1.1078865586730096; collision cylinder length=0.5885490024600376 radius=0.774072067857943; visual cylinder length=0.5885490024600376 radius=0.774072067857943
- added link 25, mass 1.1078865586730096; collision cylinder length=0.5885490024600376 radius=0.774072067857943; visual cylinder length=0.5885490024600376 radius=0.774072067857943
- link 0: mass 0.0656625499606453 -> 0.013079437091548709; geometry collision cylinder length=0.35940935990721423 radius=0.10762790799951505; visual cylinder length=0.35940935990721423 radius=0.10762790799951505
- link 11: mass 0.09777328110326605 -> 0.000346565382932485; geometry collision cylinder length=0.00014309724393646306 radius=0.878015169482812; visual cylinder length=0.00014309724393646306 radius=0.878015169482812
Joints:
- added joint 22_to_11: type revolute, parent 11, child 22, origin xyz=0.7174258218115571 0.9241630040425354 0.6345313651243545 rpy=3.187479884946322 0.5826987100304208 1.9187399681391597, axis 0 0 1, limit lower=3.1415 upper=-3.1415 effort=1 velocity=1
- added joint 23_to_11: type revolute, parent 11, child 23, origin xyz=0.7174258218115571 0.9241630040425354 0.6345313651243545 rpy=4.781219827419483 0.5826987100304208 1.9187399681391597, axis 0 0 1, limit lower=3.1415 upper=-3.1415 effort=1 velocity=1
- added joint 24_to_11: type revolute, parent 11, child 24, origin xyz=0.7174258218115571 0.9241630040425354 0.6345313651243545 rpy=6.374959769892644 0.5826987100304208 1.9187399681391597, axis 0 0 1, limit lower=3.1415 upper=-3.1415 effort=1 velocity=1
- added joint 25_to_11: type revolute, parent 11, child 25, origin xyz=0.7174258218115571 0.9241630040425354 0.6345313651243545 rpy=7.968699712365805 0.5826987100304208 1.9187399681391597, axis 0 0 1, limit lower=3.1415 upper=-3.1415 effort=1 velocity=1
- joint 11_to_0: origin xyz=0.6952506915179402 0.8815945829934303 0.4522187053142819 rpy=6.021208138471891 3.827880140251571 3.497393685292438 -> xyz=0.14857603399565733 0.850922854525532 0.8784038689011624 rpy=0.14649725603420974 4.846653697982699 5.321823417325937

File: temp4.urdf (robot description, URDF)
Before this commit: robot pepe, 8 links, 7 joints
Links:
- removed link 34
- removed link 35
- removed link 36
- removed link 37
- added link 24, mass 0.08656216894796107; collision cylinder length=0.6698241132036055 radius=0.20281904790217475; visual cylinder length=0.6698241132036055 radius=0.20281904790217475
- added link 25, mass 0.08656216894796107; collision cylinder length=0.6698241132036055 radius=0.20281904790217475; visual cylinder length=0.6698241132036055 radius=0.20281904790217475
- link 0: mass 0.0656625499606453 -> 0.013079437091548709; geometry collision cylinder length=0.35940935990721423 radius=0.10762790799951505; visual cylinder length=0.35940935990721423 radius=0.10762790799951505
- link 11: mass 0.09777328110326605 -> 0.000346565382932485; geometry collision cylinder length=0.00014309724393646306 radius=0.878015169482812; visual cylinder length=0.00014309724393646306 radius=0.878015169482812
- link 22: mass 0.357073931956523 -> 0.08656216894796107; geometry collision cylinder length=0.6698241132036055 radius=0.20281904790217475; visual cylinder length=0.6698241132036055 radius=0.20281904790217475
- link 23: mass 0.357073931956523 -> 0.08656216894796107; geometry collision cylinder length=0.6698241132036055 radius=0.20281904790217475; visual cylinder length=0.6698241132036055 radius=0.20281904790217475
Joints:
- removed joint 34_to_11
- removed joint 35_to_11
- removed joint 36_to_11
- removed joint 37_to_11
- added joint 24_to_11: type revolute, parent 11, child 24, origin xyz=0.6462597085189629 0.8247703460954684 0.3225897180783439 rpy=1.4891199591979882 2.753265867417977 0.13256535444230305, axis 0 0 1, limit lower=3.1415 upper=-3.1415 effort=1 velocity=1
- added joint 25_to_11: type revolute, parent 11, child 25, origin xyz=0.6462597085189629 0.8247703460954684 0.3225897180783439 rpy=1.8613999489974853 2.753265867417977 0.13256535444230305, axis 0 0 1, limit lower=3.1415 upper=-3.1415 effort=1 velocity=1
- joint 11_to_0: origin xyz=0.6952506915179402 0.8815945829934303 0.4522187053142819 rpy=6.021208138471891 3.827880140251571 3.497393685292438 -> xyz=0.006344866733315244 0.850922854525532 0.8784038689011624 rpy=0.14649725603420974 4.846653697982699 5.321823417325937
- joint 22_to_11: axis 0 1 0 -> 0 0 1; origin xyz=0.4629956474248542 0.15295891958123453 0.2787447681945542 rpy=3.187399433171077 3.1556927090780684 0.22993842633188863 -> xyz=0.6462597085189629 0.8247703460954684 0.3225897180783439 rpy=0.7445599795989941 2.753265867417977 0.13256535444230305
- joint 23_to_11: axis 0 1 0 -> 0 0 1; origin xyz=0.4629956474248542 0.15295891958123453 0.2787447681945542 rpy=4.781099149756615 3.1556927090780684 0.22993842633188863 -> xyz=0.6462597085189629 0.8247703460954684 0.3225897180783439 rpy=1.1168399693984912 2.753265867417977 0.13256535444230305

File: temp5.urdf (robot description, URDF)
Before this commit: robot pepe, 2 links, 1 joints
Links:
- added link 22, mass 1.1078865586730096; collision cylinder length=0.5885490024600376 radius=0.774072067857943; visual cylinder length=0.5885490024600376 radius=0.774072067857943
- link 0: mass 0.05272695044460802 -> 0.013079437091548709; geometry collision cylinder length=0.35940935990721423 radius=0.10762790799951505; visual cylinder length=0.35940935990721423 radius=0.10762790799951505
- link 11: mass 0.43893179769285917 -> 0.000346565382932485; geometry collision cylinder length=0.00014309724393646306 radius=0.878015169482812; visual cylinder length=0.00014309724393646306 radius=0.878015169482812
Joints:
- added joint 22_to_11: type revolute, parent 11, child 22, origin xyz=0.7174258218115571 0.9241630040425354 0.6345313651243545 rpy=3.187479884946322 0.5826987100304208 1.9187399681391597, axis 0 0 1, limit lower=3.1415 upper=-3.1415 effort=1 velocity=1
- joint 11_to_0: axis 0 0 1 -> 1 0 0; origin xyz=0.8317592498885846 0.6506740518234515 0.028898558806017098 rpy=4.242709261096144 6.242736811171016 1.6189296120094512 -> xyz=0.14857603399565733 0.850922854525532 0.8784038689011624 rpy=0.14649725603420974 4.846653697982699 5.321823417325937
