Commit message: update write to csv based on worksheet

File: temp6.urdf (robot description, URDF)
Before this commit: robot pepe, 13 links, 12 joints
Links:
- removed link 110
- removed link 14
- removed link 17
- removed link 211
- removed link 212
- removed link 26
- removed link 28
- removed link 29
- added link 24, mass 1.1078865586730096; collision cylinder length=0.5885490024600376 radius=0.774072067857943; visual cylinder length=0.5885490024600376 radius=0.774072067857943
- added link 36, mass 0.08656216894796107; collision cylinder length=0.6698241132036055 radius=0.20281904790217475; visual cylinder length=0.6698241132036055 radius=0.20281904790217475
- added link 37, mass 0.08656216894796107; collision cylinder length=0.6698241132036055 radius=0.20281904790217475; visual cylinder length=0.6698241132036055 radius=0.20281904790217475
- added link 38, mass 0.08656216894796107; collision cylinder length=0.6698241132036055 radius=0.20281904790217475; visual cylinder length=0.6698241132036055 radius=0.20281904790217475
- added link 39, mass 0.08656216894796107; collision cylinder length=0.6698241132036055 radius=0.20281904790217475; visual cylinder length=0.6698241132036055 radius=0.20281904790217475
- link 0: mass 0.05272695044460802 -> 0.013079437091548709; geometry collision cylinder length=0.35940935990721423 radius=0.10762790799951505; visual cylinder length=0.35940935990721423 radius=0.10762790799951505
- link 11: mass 0.6762555372256879 -> 0.000346565382932485; geometry collision cylinder length=0.00014309724393646306 radius=0.878015169482812; visual cylinder length=0.00014309724393646306 radius=0.878015169482812
- link 22: mass 0.0848987674694995 -> 1.1078865586730096; geometry collision cylinder length=0.5885490024600376 radius=0.774072067857943; visual cylinder length=0.5885490024600376 radius=0.774072067857943
- link 23: mass 0.0848987674694995 -> 1.1078865586730096; geometry collision cylinder length=0.5885490024600376 radius=0.774072067857943; visual cylinder length=0.5885490024600376 radius=0.774072067857943
- link 25: mass 0.0848987674694995 -> 1.1078865586730096; geometry collision cylinder length=0.5885490024600376 radius=0.774072067857943; visual cylinder length=0.5885490024600376 radius=0.774072067857943
Joints:
- removed joint 110_to_0
- removed joint 14_to_0
- removed joint 17_to_0
- removed joint 211_to_110
- removed joint 212_to_110
- removed joint 25_to_14
- removed joint 26_to_14
- removed joint 28_to_17
- removed joint 29_to_17
- added joint 24_to_11: type revolute, parent 11, child 24, origin xyz=0.7174258218115571 0.9241630040425354 0.6345313651243545 rpy=6.374959769892644 0.5826987100304208 1.9187399681391597, axis 0 0 1, limit lower=3.1415 upper=-3.1415 effort=1 velocity=1
- added joint 25_to_11: type revolute, parent 11, child 25, origin xyz=0.7174258218115571 0.9241630040425354 0.6345313651243545 rpy=7.968699712365805 0.5826987100304208 1.9187399681391597, axis 0 0 1, limit lower=3.1415 upper=-3.1415 effort=1 velocity=1
- added joint 36_to_11: type revolute, parent 11, child 36, origin xyz=0.6462597085189629 0.8247703460954684 0.3225897180783439 rpy=2.2336799387969823 2.753265867417977 0.13256535444230305, axis 0 0 1, limit lower=3.1415 upper=-3.1415 effort=1 velocity=1
- added joint 37_to_11: type revolute, parent 11, child 37, origin xyz=0.6462597085189629 0.8247703460954684 0.3225897180783439 rpy=2.605959928596479 2.753265867417977 0.13256535444230305, axis 0 0 1, limit lower=3.1415 upper=-3.1415 effort=1 velocity=1
- added joint 38_to_11: type revolute, parent 11, child 38, origin xyz=0.6462597085189629 0.8247703460954684 0.3225897180783439 rpy=2.9782399183959765 2.753265867417977 0.13256535444230305, axis 0 0 1, limit lower=3.1415 upper=-3.1415 effort=1 velocity=1
- added joint 39_to_11: type revolute, parent 11, child 39, origin xyz=0.6462597085189629 0.8247703460954684 0.3225897180783439 rpy=3.3505199081954737 2.753265867417977 0.13256535444230305, axis 0 0 1, limit lower=3.1415 upper=-3.1415 effort=1 velocity=1
- joint 11_to_0: axis 0 0 1 -> 1 0 0; origin xyz=0.7713827438134189 0.8471844793559141 0.7733132300909366 rpy=1.1685017951966374 2.607990398758587 5.279593793770392 -> xyz=0.14857603399565733 0.850922854525532 0.8784038689011624 rpy=0.14649725603420974 4.846653697982699 5.321823417325937
- joint 22_to_11: origin xyz=0.2185246845322868 0.7707014948884033 0.15637817477119464 rpy=11.62505959161293 0.22062271482782447 5.6968441093664515 -> xyz=0.7174258218115571 0.9241630040425354 0.6345313651243545 rpy=3.187479884946322 0.5826987100304208 1.9187399681391597
- joint 23_to_11: origin xyz=0.2185246845322868 0.7707014948884033 0.15637817477119464 rpy=17.437589387419393 0.22062271482782447 5.6968441093664515 -> xyz=0.7174258218115571 0.9241630040425354 0.6345313651243545 rpy=4.781219827419483 0.5826987100304208 1.9187399681391597

File: temp7.urdf (robot description, URDF)
Before this commit: robot pepe, 8 links, 7 joints
Links:
- removed link 22
- removed link 23
- removed link 34
- removed link 35
- removed link 36
- removed link 37
- added link 12, mass 0.02270703494692649; collision cylinder length=0.8470135737048601 radius=0.09237619993412371; visual cylinder length=0.8470135737048601 radius=0.09237619993412371
- added link 13, mass 0.02270703494692649; collision cylinder length=0.8470135737048601 radius=0.09237619993412371; visual cylinder length=0.8470135737048601 radius=0.09237619993412371
- added link 14, mass 0.02270703494692649; collision cylinder length=0.8470135737048601 radius=0.09237619993412371; visual cylinder length=0.8470135737048601 radius=0.09237619993412371
- link 0: mass 0.05272695044460802 -> 0.000346565382932485; geometry collision cylinder length=0.00014309724393646306 radius=0.878015169482812; visual cylinder length=0.00014309724393646306 radius=0.878015169482812
- link 11: mass 0.09777328110326605 -> 0.02270703494692649; geometry collision cylinder length=0.8470135737048601 radius=0.09237619993412371; visual cylinder length=0.8470135737048601 radius=0.09237619993412371
Joints:
- removed joint 22_to_11
- removed joint 23_to_11
- removed joint 34_to_0
- removed joint 35_to_0
- removed joint 36_to_0
- removed joint 37_to_0
- added joint 12_to_0: type revolute, parent 0, child 12, origin xyz=0.34167592979167816 0.7741555189693887 0.11745861032152582 rpy=10.979543912651657 0.3792176625421638 5.870559705641843, axis 0 0 1, limit lower=3.1415 upper=-3.1415 effort=1 velocity=1
- added joint 13_to_0: type revolute, parent 0, child 13, origin xyz=0.34167592979167816 0.7741555189693887 0.11745861032152582 rpy=14.639391883535543 0.3792176625421638 5.870559705641843, axis 0 0 1, limit lower=3.1415 upper=-3.1415 effort=1 velocity=1
- added joint 14_to_0: type revolute, parent 0, child 14, origin xyz=0.34167592979167816 0.7741555189693887 0.11745861032152582 rpy=18.29923985441943 0.3792176625421638 5.870559705641843, axis 0 0 1, limit lower=3.1415 upper=-3.1415 effort=1 velocity=1
- joint 11_to_0: axis 1 0 0 -> 0 0 1; origin xyz=0.6952506915179402 0.8815945829934303 0.4522187053142819 rpy=6.021208138471891 3.827880140251571 3.497393685292438 -> xyz=0.34167592979167816 0.7741555189693887 0.11745861032152582 rpy=7.319695941767772 0.3792176625421638 5.870559705641843
